Commit message: Kinect camera added

File: swarmus_ros_description/urdf/pioneer.urdf.xacro (robot description, xacro)
@@ -122,4 +122,71 @@
     <limit effort="0" velocity="0"/>
   </joint>
+  <joint name="kinect_joint" type="fixed">
+    <child link="$(arg prefix)/kinect_ros_link" />
+    <parent link="$(arg prefix)/chassis" />
+  </joint>
+  <!-- Add the remaining xacros -->
+  <link name="$(arg prefix)/kinect_ros_link">
+    <inertial>
+      <mass value="0.1"/>
+      <origin rpy="0  0  0" xyz="0  0  0"/>
+      <inertia ixx="0" ixy="0" ixz="0" iyy="0" iyz="0" izz="0"/>
+    </inertial>
+    <collision name="collision">
+      <origin rpy="0  0  0" xyz="0       0       0.03599"/>
+      <geometry>
+        <box size="0.073000 0.276000 0.072000"/>
+      </geometry>
+    </collision>
+    <visual name="visual">
+      <origin rpy="0  0  0" xyz="0       0       0.03599"/>
+      <geometry>
+        <mesh filename="package://swarmus_ros_description/models/kinect_ros/meshes/kinect.dae" scale="1.0 1.0 1.0"/>
+      </geometry>
+    </visual>
+  </link>
+  <gazebo reference="$(arg prefix)/kinect_ros_link">
+    <sensor name="camera" type="depth">
+        <update_rate>20</update_rate>
+        <camera>
+          <horizontal_fov>1.047198</horizontal_fov>
+          <image>
+            <width>640</width>
+            <height>480</height>
+            <format>R8G8B8</format>
+          </image>
+          <clip>
+            <near>0.05</near>
+            <far>3</far>
+          </clip>
+        </camera>
+        <plugin name="camera_plugin" filename="libgazebo_ros_openni_kinect.so">
+          <baseline>0.2</baseline>
+          <alwaysOn>true</alwaysOn>
+          <!-- Keep this zero, update_rate in the parent <sensor> tag
+            will control the frame rate. -->
+          <updateRate>0.0</updateRate>
+          <cameraName>camera_ir</cameraName>
+          <imageTopicName>/camera/color/image_raw</imageTopicName>
+          <cameraInfoTopicName>/camera/color/camera_info</cameraInfoTopicName>
+          <depthImageTopicName>/camera/depth/image_raw</depthImageTopicName>
+          <depthImageCameraInfoTopicName>/camera/depth/camera_info</depthImageCameraInfoTopicName>
+          <pointCloudTopicName>/camera/depth/points</pointCloudTopicName>
+          <frameName>camera_link</frameName>
+          <pointCloudCutoff>0.5</pointCloudCutoff>
+          <pointCloudCutoffMax>3.0</pointCloudCutoffMax>
+          <distortionK1>0</distortionK1>
+          <distortionK2>0</distortionK2>
+          <distortionK3>0</distortionK3>
+          <distortionT1>0</distortionT1>
+          <distortionT2>0</distortionT2>
+          <CxPrime>0</CxPrime>
+          <Cx>0</Cx>
+          <Cy>0</Cy>
+          <focalLength>0</focalLength>
+          <hackBaseline>0</hackBaseline>
+        </plugin>
+      </sensor>
+  </gazebo>
   <gazebo reference="$(arg prefix)/imu_link">
     <sensor name="imu_sensor" type="imu">

Commit message: Added lidar

File: swarmus_ros_description/urdf/pioneer.urdf.xacro (robot description, xacro)
@@ -126,5 +126,8 @@
     <parent link="$(arg prefix)/chassis" />
   </joint>
-  <!-- Add the remaining xacros -->
+  <joint name="rplidar_join" type="fixed">
+    <child link="$(arg prefix)/rplidar"/>
+    <parent link="$(arg prefix)/chassis" />
+  </joint>
   <link name="$(arg prefix)/kinect_ros_link">
     <inertial>
@@ -146,4 +149,57 @@
     </visual>
   </link>
+  <link name="$(arg prefix)/rplidar">
+    <inertial>
+      <mass value="0.1"/>
+      <origin rpy="0  0  0.35" xyz="0  0  0"/>
+      <inertia ixx="0" ixy="0" ixz="0" iyy="0" iyz="0" izz="0"/>
+    </inertial>
+    <collision name="collision">
+      <origin rpy="0  0  0" xyz="0 0 -0.0145"/>
+      <geometry>
+        <box size="0.05 0.05 0.041"/>
+      </geometry>
+    </collision>
+    <collision name="collision_top">
+      <origin rpy="0  0  0" xyz="0 0 0.0205"/>
+      <geometry>
+        <cylinder radius="0.021" length="0.029"/>
+      </geometry>
+    </collision>
+    <visual name="visual">
+      <geometry>
+        <mesh filename="package://swarmus_ros_description/models/rplidar/meshes/hokuyo.dae" scale="1.0 1.0 1.0"/>
+      </geometry>
+    </visual>
+  </link>
+<gazebo reference="$(arg prefix)/rplidar">
+      <sensor name="laser" type="ray">
+        <pose>0.01 0 0.0175 0 -0 0</pose>
+        <ray>
+          <scan>
+            <horizontal>
+              <!-- Specs from racecar's rplidar -->base_lidar
+              <samples>360</samples>
+              <resolution>1</resolution>
+              <min_angle>-3.12413907051</min_angle>
+              <max_angle>3.12413907051</max_angle>
+            </horizontal>
+          </scan>
+          <range>
+            <min>0.15</min>
+            <max>12</max>
+            <resolution>0.01</resolution>
+          </range>
+        </ray>
+        <plugin name="laser" filename="libRayPlugin.so" />
+        <plugin name="gazebo_ros_hokuyo_controller" filename="libgazebo_ros_laser.so">
+          <topicName>scan</topicName>
+          <frameName>base_laser</frameName>
+        </plugin>
+        <always_on>1</always_on>
+        <update_rate>10</update_rate>
+        <visualize>true</visualize>
+      </sensor>
+</gazebo>
   <gazebo reference="$(arg prefix)/kinect_ros_link">
     <sensor name="camera" type="depth">

Commit message: Geometry fixed of the wheels, kinect, rplidar and base_footprint

File: swarmus_ros_description/urdf/pioneer.urdf.xacro (robot description, xacro)
@@ -4,4 +4,5 @@
   <link name="$(arg prefix)/base_footprint" />
   <link name="$(arg prefix)/base_link" />
+<!-- ================================== L ==================================-->
   <link name="$(arg prefix)/chassis">
     <inertial>
@@ -11,5 +12,5 @@
     </inertial>
     <collision name="collision">
-      <origin rpy="0  0  0" xyz="0    0    0.16"/>
+      <origin rpy="0  0  0" xyz="0    0    0"/>
       <geometry>
         <box size="0.445 0.277 0.17"/>
@@ -17,5 +18,5 @@
     </collision>
     <collision name="castor_collision">
-      <origin rpy="0  0  0" xyz="-0.2   0    0.04"/>
+      <origin rpy="0  0  0" xyz="-0.2   0    -0.12"/>
       <geometry>
         <sphere radius="0.04"/>
@@ -23,5 +24,5 @@
     </collision>
     <visual name="visual">
-      <origin rpy="0  0  0" xyz="0   0   0.2"/>
+      <origin rpy="0  0  0" xyz="0   0   0.04"/>
       <geometry>
         <mesh filename="package://swarmus_ros_description/models/pioneer_swarmus/meshes/chassis.dae" scale="1.0 1.0 1.0"/>
@@ -29,5 +30,5 @@
     </visual>
     <visual name="pioneer_swarmus__castor_visual">
-      <origin rpy="0  0  0" xyz="-0.2   0    0.04"/>
+      <origin rpy="0  0  0" xyz="-0.2   0    -0.12"/>
       <geometry>
         <sphere radius="0.04"/>
@@ -42,5 +43,5 @@
     </inertial>
     <collision name="collision">
-      <origin rpy="0  0  0" xyz="0    0   -0.03"/>
+      <origin rpy="0  0  0" xyz="0    0   0"/>
       <geometry>
         <cylinder length="0.05" radius="0.11"/>
@@ -49,5 +50,5 @@
     </collision>
     <visual name="visual">
-      <origin rpy="0  0  0" xyz="0    0   -0.03"/>
+      <origin rpy="0  0  0" xyz="0    0   0"/>
       <geometry>
         <cylinder length="0.05" radius="0.11"/>
@@ -62,5 +63,5 @@
     </inertial>
     <collision name="collision">
-      <origin rpy="0  0  0" xyz="0    0    0.03"/>
+      <origin rpy="0  0  0" xyz="0    0   0"/>
       <geometry>
         <cylinder length="0.05" radius="0.11"/>
@@ -69,5 +70,5 @@
     </collision>
     <visual name="visual">
-      <origin rpy="0  0  0" xyz="0    0    0.03"/>
+      <origin rpy="0  0  0" xyz="0    0   0"/>
       <geometry>
         <cylinder length="0.05" radius="0.11"/>
@@ -89,7 +90,51 @@
     <!-- Rajouter le sensor-->
   </link>
+  <link name="$(arg prefix)/kinect_ros_link">
+    <inertial>
+      <mass value="0.1"/>
+      <origin rpy="0  0  0" xyz="0  0  0"/>
+      <inertia ixx="0" ixy="0" ixz="0" iyy="0" iyz="0" izz="0"/>
+    </inertial>
+    <collision name="collision">
+      <origin rpy="0  0  0" xyz="0       0       0.03599"/>
+      <geometry>
+        <box size="0.073000 0.276000 0.072000"/>
+      </geometry>
+    </collision>
+    <visual name="visual">
+      <origin rpy="0  0  0" xyz="0       0       0.03599"/>
+      <geometry>
+        <mesh filename="package://swarmus_ros_description/models/kinect_ros/meshes/kinect.dae" scale="1.0 1.0 1.0"/>
+      </geometry>
+    </visual>
+  </link>
+  <link name="$(arg prefix)/rplidar">
+    <inertial>
+      <mass value="0.1"/>
+      <origin rpy="0  0  0" xyz="0  0  0"/>
+      <inertia ixx="0" ixy="0" ixz="0" iyy="0" iyz="0" izz="0"/>
+    </inertial>
+    <collision name="collision">
+      <origin rpy="0  0  0" xyz="0 0 -0.0145"/>
+      <geometry>
+        <box size="0.05 0.05 0.041"/>
+      </geometry>
+    </collision>
+    <collision name="collision_top">
+      <origin rpy="0  0  0" xyz="0 0 0.0205"/>
+      <geometry>
+        <cylinder radius="0.021" length="0.029"/>
+      </geometry>
+    </collision>
+    <visual name="visual">
+      <geometry>
+        <mesh filename="package://swarmus_ros_description/models/rplidar/meshes/hokuyo.dae" scale="1.0 1.0 1.0"/>
+      </geometry>
+    </visual>
+  </link>
+<!-- ================================== Joints ==================================-->
   <joint name="base_footprint_link_joint" type="fixed">
     <!-- The 0.5 should be changed to have the real offset from the floor-->
-    <origin xyz="0 0 0.05" rpy="0 0 0" />
+    <origin xyz="0 0 0.16" rpy="0 0 0" />
     <parent link="$(arg prefix)/base_footprint" />
     <child link="$(arg prefix)/base_link" />
@@ -104,5 +149,5 @@
     <parent link="$(arg prefix)/chassis"/>
     <child link="$(arg prefix)/left_wheel"/>
-    <origin rpy="0      1.5707  1.5707" xyz="0.1  0.14     0.11"/>
+    <origin rpy="0      1.5707  1.5707" xyz="0.1  0.17    -0.05"/>
     <axis xyz="9.00000000e-05   9.00000000e-05   1.00000000e+00"/>
     <limit effort="0.0" velocity="0.0"/>>
@@ -111,5 +156,5 @@
     <parent link="$(arg prefix)/chassis"/>
     <child link="$(arg prefix)/right_wheel"/>
-    <origin rpy="0      1.5707  1.5707" xyz="0.1  -0.14  0.11"/>
+    <origin rpy="0      1.5707  1.5707" xyz="0.1  -0.17  -0.05"/>
     <axis xyz="9.00000000e-05   9.00000000e-05   1.00000000e+00"/>
     <limit effort="0.0" velocity="0.0"/>
@@ -118,5 +163,5 @@
     <parent link="$(arg prefix)/chassis"/>
     <child link="$(arg prefix)/imu_link"/>
-    <origin rpy="0  0  0" xyz="0.07  0    0.27"/>
+    <origin rpy="0  0  0" xyz="0.07  0    0.11"/>
     <axis xyz="0  0  0"/>
     <limit effort="0" velocity="0"/>
@@ -125,52 +170,12 @@
     <child link="$(arg prefix)/kinect_ros_link" />
     <parent link="$(arg prefix)/chassis" />
-  </joint>
-  <joint name="rplidar_join" type="fixed">
+    <origin rpy="0  0  0" xyz="0.20  0    0.11"/>
+  </joint>
+  <joint name="rplidar_joint" type="fixed">
     <child link="$(arg prefix)/rplidar"/>
     <parent link="$(arg prefix)/chassis" />
-  </joint>
-  <link name="$(arg prefix)/kinect_ros_link">
-    <inertial>
-      <mass value="0.1"/>
-      <origin rpy="0  0  0" xyz="0  0  0"/>
-      <inertia ixx="0" ixy="0" ixz="0" iyy="0" iyz="0" izz="0"/>
-    </inertial>
-    <collision name="collision">
-      <origin rpy="0  0  0" xyz="0       0       0.03599"/>
-      <geometry>
-        <box size="0.073000 0.276000 0.072000"/>
-      </geometry>
-    </collision>
-    <visual name="visual">
-      <origin rpy="0  0  0" xyz="0       0       0.03599"/>
-      <geometry>
-        <mesh filename="package://swarmus_ros_description/models/kinect_ros/meshes/kinect.dae" scale="1.0 1.0 1.0"/>
-      </geometry>
-    </visual>
-  </link>
-  <link name="$(arg prefix)/rplidar">
-    <inertial>
-      <mass value="0.1"/>
-      <origin rpy="0  0  0.35" xyz="0  0  0"/>
-      <inertia ixx="0" ixy="0" ixz="0" iyy="0" iyz="0" izz="0"/>
-    </inertial>
-    <collision name="collision">
-      <origin rpy="0  0  0" xyz="0 0 -0.0145"/>
-      <geometry>
-        <box size="0.05 0.05 0.041"/>
-      </geometry>
-    </collision>
-    <collision name="collision_top">
-      <origin rpy="0  0  0" xyz="0 0 0.0205"/>
-      <geometry>
-        <cylinder radius="0.021" length="0.029"/>
-      </geometry>
-    </collision>
-    <visual name="visual">
-      <geometry>
-        <mesh filename="package://swarmus_ros_description/models/rplidar/meshes/hokuyo.dae" scale="1.0 1.0 1.0"/>
-      </geometry>
-    </visual>
-  </link>
+    <origin rpy="0  0  0" xyz="0  0    0.21"/>
+  </joint>
+<!-- ================================== Gazebo plugin ================================== -->
 <gazebo reference="$(arg prefix)/rplidar">
       <sensor name="laser" type="ray">

Commit message: Ros control added to the urdf, controller .yaml created, added ros_control joint_state_publisher and joint_controller dependancies in package .xml, transmission added to the .urdf, name prefix added in front of camera topics and deleted the pioneer_semi_completed.urdf since it was a temp file

File: swarmus_ros_description/urdf/pioneer.urdf.xacro (robot description, xacro)
@@ -47,5 +47,4 @@
         <cylinder length="0.05" radius="0.11"/>
       </geometry>
-      <!-- pas de friction?-->
     </collision>
     <visual name="visual">
@@ -67,5 +66,4 @@
         <cylinder length="0.05" radius="0.11"/>
       </geometry>
-      <!-- pas de friction?-->
     </collision>
     <visual name="visual">
@@ -88,5 +86,4 @@
       </geometry>
     </visual>
-    <!-- Rajouter le sensor-->
   </link>
   <link name="$(arg prefix)/kinect_ros_link">
@@ -135,5 +132,4 @@
 <!-- ================================== Joints ==================================-->
   <joint name="base_footprint_link_joint" type="fixed">
-    <!-- The 0.5 should be changed to have the real offset from the floor-->
     <origin xyz="0 0 0.16" rpy="0 0 0" />
     <parent link="$(arg prefix)/base_footprint" />
@@ -141,5 +137,4 @@
   </joint>
   <joint name="base_link_chassis_joint" type="fixed">
-    <!-- The 0.5 should be changed to have the real offset from the floor-->
     <origin xyz="0 0 0.0" rpy="0 0 0" />
     <parent link="$(arg prefix)/base_link" />
@@ -178,5 +173,55 @@
   </joint>
 <!-- ================================== Gazebo plugin ================================== -->
-<gazebo reference="$(arg prefix)/rplidar">
+<gazebo reference="$(arg prefix)/chassis">
+  <mu1 value="0.0"/>
+  <mu2 value="0.0"/>
+  <kp  value="1.0" />
+  <kd  value="1.0" />
+  <!-- material>Gazebo/$(arg color)</material-->
+</gazebo>
+<gazebo reference="$(arg prefix)/right_wheel">
+  <mu1 value="100000.0"/>
+  <mu2 value="100000.0"/>
+  <kp  value="0.0" />
+  <kd  value="0.0" />
+  <!-- material>Gazebo/$(arg color)</material-->
+</gazebo>
+<gazebo reference="$(arg prefix)/left_wheel">
+  <mu1 value="100000.0"/>
+  <mu2 value="100000.0"/>
+  <kp  value="0.0" />
+  <kd  value="0.0" />
+  <!-- material>Gazebo/$(arg color)</material-->
+</gazebo>
+<gazebo>
+  <plugin name="gazebo_ros_control" filename="libgazebo_ros_control.so">
+    <robotNamespace>$(arg prefix)</robotNamespace>
+    <robotSimType>gazebo_ros_control/DefaultRobotHWSim</robotSimType>
+  </plugin>
+</gazebo>
+  <gazebo>
+    <plugin name="differential_drive" filename="libgazebo_ros_diff_drive.so">
+      <robotNamespace>$(arg prefix)</robotNamespace>
+      <commandTopic>cmd_vel</commandTopic>
+      <odometryTopic>odom</odometryTopic>
+      <odometryFrame>odom</odometryFrame>
+      <odometrySource>world</odometrySource>
+      <publishOdomTF>true</publishOdomTF>
+      <robotBaseFrame>$(arg prefix)/base_footprint</robotBaseFrame>
+      <publishWheelTF>false</publishWheelTF>
+      <publishTf>true</publishTf>
+      <publishWheelJointState>true</publishWheelJointState>
+      <legacyMode>false</legacyMode>
+      <updateRate>50</updateRate>
+      <leftJoint>$(arg prefix)/left_wheel</leftJoint>
+      <rightJoint>$(arg prefix)/right_wheel</rightJoint>
+      <wheelSeparation>0.34</wheelSeparation>
+      <wheelDiameter>0.22</wheelDiameter>
+      <wheelAcceleration>1</wheelAcceleration>
+      <wheelTorque>10</wheelTorque>
+      <rosDebugLevel>na</rosDebugLevel>
+    </plugin>
+  </gazebo>
+  <gazebo reference="$(arg prefix)/rplidar">
       <sensor name="laser" type="ray">
         <pose>0.01 0 0.0175 0 -0 0</pose>
@@ -199,4 +244,5 @@
         <plugin name="laser" filename="libRayPlugin.so" />
         <plugin name="gazebo_ros_hokuyo_controller" filename="libgazebo_ros_laser.so">
+          <robotNamespace>$(arg prefix)</robotNamespace>
           <topicName>scan</topicName>
           <frameName>base_laser</frameName>
@@ -206,5 +252,5 @@
         <visualize>true</visualize>
       </sensor>
-</gazebo>
+  </gazebo>
   <gazebo reference="$(arg prefix)/kinect_ros_link">
     <sensor name="camera" type="depth">
@@ -223,4 +269,5 @@
         </camera>
         <plugin name="camera_plugin" filename="libgazebo_ros_openni_kinect.so">
+          <robotNamespace>$(arg prefix)</robotNamespace>
           <baseline>0.2</baseline>
           <alwaysOn>true</alwaysOn>
@@ -229,9 +276,9 @@
           <updateRate>0.0</updateRate>
           <cameraName>camera_ir</cameraName>
-          <imageTopicName>/camera/color/image_raw</imageTopicName>
+          <!--imageTopicName>/camera/color/image_raw</imageTopicName>
           <cameraInfoTopicName>/camera/color/camera_info</cameraInfoTopicName>
           <depthImageTopicName>/camera/depth/image_raw</depthImageTopicName>
           <depthImageCameraInfoTopicName>/camera/depth/camera_info</depthImageCameraInfoTopicName>
-          <pointCloudTopicName>/camera/depth/points</pointCloudTopicName>
+          <pointCloudTopicName>/camera/depth/points</pointCloudTopicName-->
           <frameName>camera_link</frameName>
           <pointCloudCutoff>0.5</pointCloudCutoff>
@@ -253,4 +300,5 @@
     <sensor name="imu_sensor" type="imu">
       <plugin filename="libgazebo_ros_imu_sensor.so" name="imu_plugin">
+        <robotNamespace>$(arg prefix)</robotNamespace>
         <topicName>imu/data</topicName>
         <bodyName>$(arg prefix)/imu_link</bodyName>
@@ -263,3 +311,22 @@
     </sensor>
   </gazebo>
+<!-- ================================== Transmission ================================== -->
+  <transmission name="$(arg prefix)_right_wheel_trans">
+    <type>transmission_interface/SimpleTransmission</type>
+    <actuator name="$(arg prefix)_right_wheel_motor">
+      <mechanicalReduction>1</mechanicalReduction>
+    </actuator>
+    <joint name="right_wheel_hinge">
+      <hardwareInterface>hardware_interface/EffortJointInterface</hardwareInterface>
+    </joint>
+  </transmission>
+  <transmission name="$(arg prefix)_left_wheel_trans">
+    <type>transmission_interface/SimpleTransmission</type>
+    <actuator name="$(arg prefix)_left_wheel_motor">
+      <mechanicalReduction>1</mechanicalReduction>
+    </actuator>
+    <joint name="left_wheel_hinge">
+      <hardwareInterface>hardware_interface/EffortJointInterface</hardwareInterface>
+    </joint>
+  </transmission>
 </robot>

Commit message: Hiveboard box added in the .URDF

File: swarmus_ros_description/urdf/pioneer.urdf.xacro (robot description, xacro)
@@ -130,4 +130,20 @@
     </visual>
   </link>
+  <link name="$(arg prefix)/hiveboard">
+    <inertial>
+      <mass value="0.0000001"/>
+      <origin rpy="0  0  0" xyz="0  0  0"/>
+      <inertia ixx="0.00001" ixy="0" ixz="0" iyy="0.00001" iyz="0" izz="0.00001"/>
+    </inertial>
+    <visual name="visual">
+      <origin rpy="0  0  0" xyz="0  0  0"/>
+      <geometry>
+        <box size="0.07 0.07 0.02"/>
+      </geometry>
+      <material name="Orange">
+        <color rgba="1.0 0.622 0.0 1"/>
+      </material>
+    </visual>
+  </link>
 <!-- ================================== Joints ==================================-->
   <joint name="base_footprint_link_joint" type="fixed">
@@ -171,4 +187,9 @@
     <parent link="$(arg prefix)/chassis" />
     <origin rpy="0  0  0" xyz="0  0    0.21"/>
+  </joint>
+  <joint name="hiveboard_joint" type="fixed">
+    <child link="$(arg prefix)/hiveboard"/>
+    <parent link="$(arg prefix)/chassis"/>
+    <origin rpy="0  0  0" xyz="-0.1  0.0  0.12"/>
   </joint>
 <!-- ================================== Gazebo plugin ================================== -->

Commit message: Removed movement limitation / set to speed control
Controller can now be controlled by settings up their velocity thorugh the controller command.

File: swarmus_ros_description/urdf/pioneer.urdf.xacro (robot description, xacro)
@@ -162,5 +162,5 @@
     <origin rpy="0      1.5707  1.5707" xyz="0.1  0.17    -0.05"/>
     <axis xyz="9.00000000e-05   9.00000000e-05   1.00000000e+00"/>
-    <limit effort="0.0" velocity="0.0"/>>
+    <limit effort="100.0" velocity="100"/>>
   </joint>
   <joint name="right_wheel_hinge" type="continuous">
@@ -169,5 +169,5 @@
     <origin rpy="0      1.5707  1.5707" xyz="0.1  -0.17  -0.05"/>
     <axis xyz="9.00000000e-05   9.00000000e-05   1.00000000e+00"/>
-    <limit effort="0.0" velocity="0.0"/>
+    <limit effort="100.0" velocity="100"/>
   </joint>
   <joint name="imu_joint" type="fixed">
@@ -217,5 +217,5 @@
 <gazebo>
   <plugin name="gazebo_ros_control" filename="libgazebo_ros_control.so">
-    <robotSimType>gazebo_ros_control/DefaultRobotHWSim</robotSimType>
+    <!--robotSimType>gazebo_ros_control/DefaultRobotHWSim</robotSimType-->
   </plugin>
 </gazebo>

Commit message: Controllers config changes

File: swarmus_ros_description/urdf/pioneer.urdf.xacro (robot description, xacro)
@@ -162,5 +162,5 @@
     <origin rpy="0      1.5707  1.5707" xyz="0.1  0.17    -0.05"/>
     <axis xyz="9.00000000e-05   9.00000000e-05   1.00000000e+00"/>
-    <limit effort="100.0" velocity="100"/>>
+    <limit effort="100.0" velocity="100"/>
   </joint>
   <joint name="right_wheel_hinge" type="continuous">
@@ -270,5 +270,5 @@
         <always_on>1</always_on>
         <update_rate>10</update_rate>
-        <visualize>true</visualize>
+        <visualize>false</visualize>
       </sensor>
   </gazebo>
