Commit message: Fixed the odometry publishing. Remove the joint_state_controller transmission because the odometry plugin has a built differential controller easier to use. Changed the child link of the tf_publisher for /odom since the odomertry plugin publish a tf between /odom and base_footprint

File: swarmus_ros_description/urdf/pioneer.urdf.xacro (robot description, xacro)
@@ -222,5 +222,5 @@
   <gazebo>
     <plugin name="differential_drive" filename="libgazebo_ros_diff_drive.so">
-      <robotNamespace>$(arg prefix)</robotNamespace>
+      <!--robotNamespace>$(arg prefix)</robotNamespace-->
       <commandTopic>cmd_vel</commandTopic>
       <odometryTopic>odom</odometryTopic>
@@ -228,5 +228,5 @@
       <odometrySource>world</odometrySource>
       <publishOdomTF>true</publishOdomTF>
-      <robotBaseFrame>$(arg prefix)/base_footprint</robotBaseFrame>
+      <robotBaseFrame>base_footprint</robotBaseFrame>
       <publishWheelTF>false</publishWheelTF>
       <publishTf>true</publishTf>
@@ -234,11 +234,11 @@
       <legacyMode>false</legacyMode>
       <updateRate>50</updateRate>
-      <leftJoint>$(arg prefix)/left_wheel</leftJoint>
-      <rightJoint>$(arg prefix)/right_wheel</rightJoint>
+      <leftJoint>left_wheel_hinge</leftJoint>
+      <rightJoint>right_wheel_hinge</rightJoint>
       <wheelSeparation>0.34</wheelSeparation>
       <wheelDiameter>0.22</wheelDiameter>
       <wheelAcceleration>1</wheelAcceleration>
       <wheelTorque>10</wheelTorque>
-      <rosDebugLevel>na</rosDebugLevel>
+      <rosDebugLevel>true</rosDebugLevel>
     </plugin>
   </gazebo>
@@ -331,22 +331,3 @@
     </sensor>
   </gazebo>
-<!-- ================================== Transmission ================================== -->
-  <transmission name="$(arg prefix)_right_wheel_trans">
-    <type>transmission_interface/SimpleTransmission</type>
-    <actuator name="$(arg prefix)_right_wheel_motor">
-      <mechanicalReduction>1</mechanicalReduction>
-    </actuator>
-    <joint name="right_wheel_hinge">
-      <hardwareInterface>hardware_interface/EffortJointInterface</hardwareInterface>
-    </joint>
-  </transmission>
-  <transmission name="$(arg prefix)_left_wheel_trans">
-    <type>transmission_interface/SimpleTransmission</type>
-    <actuator name="$(arg prefix)_left_wheel_motor">
-      <mechanicalReduction>1</mechanicalReduction>
-    </actuator>
-    <joint name="left_wheel_hinge">
-      <hardwareInterface>hardware_interface/EffortJointInterface</hardwareInterface>
-    </joint>
-  </transmission>
 </robot>

Commit message: Changed the directory of the meshes to be more close to root. Deleted the models directory since it's now useless

File: swarmus_ros_description/urdf/pioneer.urdf.xacro (robot description, xacro)
@@ -26,5 +26,5 @@
       <origin rpy="0  0  0" xyz="0   0   0.04"/>
       <geometry>
-        <mesh filename="package://swarmus_ros_description/models/pioneer_swarmus/meshes/chassis.dae" scale="1.0 1.0 1.0"/>
+        <mesh filename="package://swarmus_ros_description/meshes/chassis.dae" scale="1.0 1.0 1.0"/>
       </geometry>
     </visual>
@@ -102,5 +102,5 @@
       <origin rpy="0  0  0" xyz="0       0       0.03599"/>
       <geometry>
-        <mesh filename="package://swarmus_ros_description/models/kinect_ros/meshes/kinect.dae" scale="1.0 1.0 1.0"/>
+        <mesh filename="package://swarmus_ros_description/meshes/kinect.dae" scale="1.0 1.0 1.0"/>
       </geometry>
     </visual>
@@ -126,5 +126,5 @@
     <visual name="visual">
       <geometry>
-        <mesh filename="package://swarmus_ros_description/models/rplidar/meshes/hokuyo.dae" scale="1.0 1.0 1.0"/>
+        <mesh filename="package://swarmus_ros_description/meshes/hokuyo.dae" scale="1.0 1.0 1.0"/>
       </geometry>
     </visual>

Commit message: Changed castor for caster in the URDF

File: swarmus_ros_description/urdf/pioneer.urdf.xacro (robot description, xacro)
@@ -17,5 +17,5 @@
       </geometry>
     </collision>
-    <collision name="castor_collision">
+    <collision name="caster_collision">
       <origin rpy="0  0  0" xyz="-0.2   0    -0.12"/>
       <geometry>
@@ -29,5 +29,5 @@
       </geometry>
     </visual>
-    <visual name="pioneer_swarmus__castor_visual">
+    <visual name="caster_visual">
       <origin rpy="0  0  0" xyz="-0.2   0    -0.12"/>
       <geometry>

Commit message: PR fixes
[SWARINFO-47] Add communication and interlocalization for simulated HiveBoard #2

File: swarmus_ros_description/urdf/pioneer.urdf.xacro (robot description, xacro)
@@ -1,16 +1,17 @@
 <?xml version="1.0" ?>
-<robot name="pioneer_swarmus" xmlns:xacro="http://www.ros.org/wiki/xacro">
+<robot name="pioneer_swarmus"
+  xmlns:xacro="http://www.ros.org/wiki/xacro">
   <xacro:arg name="prefix" default="p_swarmus"/>
   <link name="$(arg prefix)/base_footprint" />
   <link name="$(arg prefix)/base_link" />
-<!-- ================================== Links ==================================-->
+  <!-- ================================== Links ==================================-->
   <link name="$(arg prefix)/chassis">
     <inertial>
       <mass value="5.67"/>
-      <origin rpy="0  0  0" xyz="0  0  0"/>
+      <origin rpy="0 0 0" xyz="0 0 0"/>
       <inertia ixx="0.07" ixy="0" ixz="0" iyy="0.08" iyz="0" izz="0.10"/>
     </inertial>
     <collision name="collision">
-      <origin rpy="0  0  0" xyz="0    0    0"/>
+      <origin rpy="0 0 0" xyz="0 0 0"/>
       <geometry>
         <box size="0.445 0.277 0.17"/>
@@ -18,5 +19,5 @@
     </collision>
     <collision name="castor_collision">
-      <origin rpy="0  0  0" xyz="-0.2   0    -0.12"/>
+      <origin rpy="0 0 0" xyz="-0.2 0 -0.12"/>
       <geometry>
         <sphere radius="0.04"/>
@@ -24,5 +25,5 @@
     </collision>
     <visual name="visual">
-      <origin rpy="0  0  0" xyz="0   0   0.04"/>
+      <origin rpy="0 0 0" xyz="0 0 0.04"/>
       <geometry>
         <mesh filename="package://swarmus_ros_description/models/pioneer_swarmus/meshes/chassis.dae" scale="1.0 1.0 1.0"/>
@@ -30,5 +31,5 @@
     </visual>
     <visual name="pioneer_swarmus__castor_visual">
-      <origin rpy="0  0  0" xyz="-0.2   0    -0.12"/>
+      <origin rpy="0 0 0" xyz="-0.2 0 -0.12"/>
       <geometry>
         <sphere radius="0.04"/>
@@ -39,9 +40,9 @@
     <inertial>
       <mass value="1.5"/>
-      <origin rpy="0  0  0" xyz="0  0  0"/>
+      <origin rpy="0 0 0" xyz="0 0 0"/>
       <inertia ixx="0.0051" ixy="0" ixz="0" iyy="0.0051" iyz="0" izz="0.0090"/>
     </inertial>
     <collision name="collision">
-      <origin rpy="0  0  0" xyz="0    0   0"/>
+      <origin rpy="0 0 0" xyz="0 0 0"/>
       <geometry>
         <cylinder length="0.05" radius="0.11"/>
@@ -49,5 +50,5 @@
     </collision>
     <visual name="visual">
-      <origin rpy="0  0  0" xyz="0    0   0"/>
+      <origin rpy="0 0 0" xyz="0 0 0"/>
       <geometry>
         <cylinder length="0.05" radius="0.11"/>
@@ -58,9 +59,9 @@
     <inertial>
       <mass value="1.5"/>
-      <origin rpy="0  0  0" xyz="0  0  0"/>
+      <origin rpy="0 0 0" xyz="0 0 0"/>
       <inertia ixx="0.0051" ixy="0" ixz="0" iyy="0.0051" iyz="0" izz="0.0090"/>
     </inertial>
     <collision name="collision">
-      <origin rpy="0  0  0" xyz="0    0   0"/>
+      <origin rpy="0 0 0" xyz="0 0 0"/>
       <geometry>
         <cylinder length="0.05" radius="0.11"/>
@@ -68,5 +69,5 @@
     </collision>
     <visual name="visual">
-      <origin rpy="0  0  0" xyz="0    0   0"/>
+      <origin rpy="0 0 0" xyz="0 0 0"/>
       <geometry>
         <cylinder length="0.05" radius="0.11"/>
@@ -77,9 +78,9 @@
     <inertial>
       <mass value="0.0000001"/>
-      <origin rpy="0  0  0" xyz="0  0  0"/>
+      <origin rpy="0 0 0" xyz="0 0 0"/>
       <inertia ixx="0.00001" ixy="0" ixz="0" iyy="0.00001" iyz="0" izz="0.00001"/>
     </inertial>
     <visual name="pioneer_swarmus__visual">
-      <origin rpy="0  0  0" xyz="0  0  0"/>
+      <origin rpy="0 0 0" xyz="0 0 0"/>
       <geometry>
         <box size="0.03 0.03 0.01"/>
@@ -90,9 +91,9 @@
     <inertial>
       <mass value="0.1"/>
-      <origin rpy="0  0  0" xyz="0  0  0"/>
+      <origin rpy="0 0 0" xyz="0 0 0"/>
       <inertia ixx="0" ixy="0" ixz="0" iyy="0" iyz="0" izz="0"/>
     </inertial>
     <collision name="collision">
-      <origin rpy="0  0  0" xyz="0       0       0.03599"/>
+      <origin rpy="0 0 0" xyz="0 0 0.03599"/>
       <geometry>
         <box size="0.073000 0.276000 0.072000"/>
@@ -100,5 +101,5 @@
     </collision>
     <visual name="visual">
-      <origin rpy="0  0  0" xyz="0       0       0.03599"/>
+      <origin rpy="0 0 0" xyz="0 0 0.03599"/>
       <geometry>
         <mesh filename="package://swarmus_ros_description/models/kinect_ros/meshes/kinect.dae" scale="1.0 1.0 1.0"/>
@@ -109,9 +110,9 @@
     <inertial>
       <mass value="0.1"/>
-      <origin rpy="0  0  0" xyz="0  0  0"/>
+      <origin rpy="0 0 0" xyz="0 0 0"/>
       <inertia ixx="0" ixy="0" ixz="0" iyy="0" iyz="0" izz="0"/>
     </inertial>
     <collision name="collision">
-      <origin rpy="0  0  0" xyz="0 0 -0.0145"/>
+      <origin rpy="0 0 0" xyz="0 0 -0.0145"/>
       <geometry>
         <box size="0.05 0.05 0.041"/>
@@ -119,5 +120,5 @@
     </collision>
     <collision name="collision_top">
-      <origin rpy="0  0  0" xyz="0 0 0.0205"/>
+      <origin rpy="0 0 0" xyz="0 0 0.0205"/>
       <geometry>
         <cylinder radius="0.021" length="0.029"/>
@@ -133,9 +134,9 @@
     <inertial>
       <mass value="0.0000001"/>
-      <origin rpy="0  0  0" xyz="0  0  0"/>
+      <origin rpy="0 0 0" xyz="0 0 0"/>
       <inertia ixx="0.00001" ixy="0" ixz="0" iyy="0.00001" iyz="0" izz="0.00001"/>
     </inertial>
     <visual name="visual">
-      <origin rpy="0  0  0" xyz="0  0  0"/>
+      <origin rpy="0 0 0" xyz="0 0 0"/>
       <geometry>
         <box size="0.07 0.07 0.02"/>
@@ -146,5 +147,5 @@
     </visual>
   </link>
-<!-- ================================== Joints ==================================-->
+  <!-- ================================== Joints ==================================-->
   <joint name="base_footprint_link_joint" type="fixed">
     <origin xyz="0 0 0.16" rpy="0 0 0" />
@@ -160,13 +161,14 @@
     <parent link="$(arg prefix)/chassis"/>
     <child link="$(arg prefix)/left_wheel"/>
-    <origin rpy="0      1.5707  1.5707" xyz="0.1  0.17    -0.05"/>
-    <axis xyz="9.00000000e-05   9.00000000e-05   1.00000000e+00"/>
-    <limit effort="0.0" velocity="0.0"/>>
+    <origin rpy="0 1.5707 1.5707" xyz="0.1 0.17 -0.05"/>
+    <axis xyz="9.00000000e-05 9.00000000e-05 1.00000000e+00"/>
+    <limit effort="0.0" velocity="0.0"/>
+>
   </joint>
   <joint name="right_wheel_hinge" type="continuous">
     <parent link="$(arg prefix)/chassis"/>
     <child link="$(arg prefix)/right_wheel"/>
-    <origin rpy="0      1.5707  1.5707" xyz="0.1  -0.17  -0.05"/>
-    <axis xyz="9.00000000e-05   9.00000000e-05   1.00000000e+00"/>
+    <origin rpy="0 1.5707 1.5707" xyz="0.1 -0.17 -0.05"/>
+    <axis xyz="9.00000000e-05 9.00000000e-05 1.00000000e+00"/>
     <limit effort="0.0" velocity="0.0"/>
   </joint>
@@ -174,6 +176,6 @@
     <parent link="$(arg prefix)/chassis"/>
     <child link="$(arg prefix)/imu_link"/>
-    <origin rpy="0  0  0" xyz="0.07  0    0.11"/>
-    <axis xyz="0  0  0"/>
+    <origin rpy="0 0 0" xyz="0.07 0 0.11"/>
+    <axis xyz="0 0 0"/>
     <limit effort="0" velocity="0"/>
   </joint>
@@ -181,43 +183,43 @@
     <child link="$(arg prefix)/kinect_ros_link" />
     <parent link="$(arg prefix)/chassis" />
-    <origin rpy="0  0  0" xyz="0.20  0    0.11"/>
+    <origin rpy="0 0 0" xyz="0.20 0 0.11"/>
   </joint>
   <joint name="rplidar_joint" type="fixed">
     <child link="$(arg prefix)/rplidar"/>
     <parent link="$(arg prefix)/chassis" />
-    <origin rpy="0  0  0" xyz="0  0    0.21"/>
+    <origin rpy="0 0 0" xyz="0 0 0.21"/>
   </joint>
   <joint name="hiveboard_joint" type="fixed">
     <child link="$(arg prefix)/hiveboard"/>
     <parent link="$(arg prefix)/chassis"/>
-    <origin rpy="0  0  0" xyz="-0.1  0.0  0.12"/>
-  </joint>
-<!-- ================================== Gazebo plugin ================================== -->
-<gazebo reference="$(arg prefix)/chassis">
-  <mu1 value="0.0"/>
-  <mu2 value="0.0"/>
-  <kp  value="1.0" />
-  <kd  value="1.0" />
-  <!-- material>Gazebo/$(arg color)</material-->
-</gazebo>
-<gazebo reference="$(arg prefix)/right_wheel">
-  <mu1 value="100000.0"/>
-  <mu2 value="100000.0"/>
-  <kp  value="0.0" />
-  <kd  value="0.0" />
-  <!-- material>Gazebo/$(arg color)</material-->
-</gazebo>
-<gazebo reference="$(arg prefix)/left_wheel">
-  <mu1 value="100000.0"/>
-  <mu2 value="100000.0"/>
-  <kp  value="0.0" />
-  <kd  value="0.0" />
-  <!-- material>Gazebo/$(arg color)</material-->
-</gazebo>
-<gazebo>
-  <plugin name="gazebo_ros_control" filename="libgazebo_ros_control.so">
-    <robotSimType>gazebo_ros_control/DefaultRobotHWSim</robotSimType>
-  </plugin>
-</gazebo>
+    <origin rpy="0 0 0" xyz="-0.1 0.0 0.12"/>
+  </joint>
+  <!-- ================================== Gazebo plugin ================================== -->
+  <gazebo reference="$(arg prefix)/chassis">
+    <mu1 value="0.0"/>
+    <mu2 value="0.0"/>
+    <kp value="1.0" />
+    <kd value="1.0" />
+    <!-- material>Gazebo/$(arg color)</material-->
+  </gazebo>
+  <gazebo reference="$(arg prefix)/right_wheel">
+    <mu1 value="100000.0"/>
+    <mu2 value="100000.0"/>
+    <kp value="0.0" />
+    <kd value="0.0" />
+    <!-- material>Gazebo/$(arg color)</material-->
+  </gazebo>
+  <gazebo reference="$(arg prefix)/left_wheel">
+    <mu1 value="100000.0"/>
+    <mu2 value="100000.0"/>
+    <kp value="0.0" />
+    <kd value="0.0" />
+    <!-- material>Gazebo/$(arg color)</material-->
+  </gazebo>
+  <gazebo>
+    <plugin name="gazebo_ros_control" filename="libgazebo_ros_control.so">
+      <robotSimType>gazebo_ros_control/DefaultRobotHWSim</robotSimType>
+    </plugin>
+  </gazebo>
   <gazebo>
     <plugin name="differential_drive" filename="libgazebo_ros_diff_drive.so">
@@ -244,76 +246,76 @@
   </gazebo>
   <gazebo reference="$(arg prefix)/rplidar">
-      <sensor name="laser" type="ray">
-        <pose>0.01 0 0.0175 0 -0 0</pose>
-        <ray>
-          <scan>
-            <horizontal>
-              <!-- Specs from racecar's rplidar -->base_lidar
-              <samples>360</samples>
-              <resolution>1</resolution>
-              <min_angle>-3.12413907051</min_angle>
-              <max_angle>3.12413907051</max_angle>
-            </horizontal>
-          </scan>
-          <range>
-            <min>0.15</min>
-            <max>12</max>
-            <resolution>0.01</resolution>
-          </range>
-        </ray>
-        <plugin name="laser" filename="libRayPlugin.so" />
-        <plugin name="gazebo_ros_hokuyo_controller" filename="libgazebo_ros_laser.so">
-          <robotNamespace>$(arg prefix)</robotNamespace>
-          <topicName>scan</topicName>
-          <frameName>base_laser</frameName>
-        </plugin>
-        <always_on>1</always_on>
-        <update_rate>10</update_rate>
-        <visualize>true</visualize>
-      </sensor>
+    <sensor name="laser" type="ray">
+      <pose>0.01 0 0.0175 0 -0 0</pose>
+      <ray>
+        <scan>
+          <horizontal>
+            <!-- Specs from racecar's rplidar -->base_lidar
+            <samples>360</samples>
+            <resolution>1</resolution>
+            <min_angle>-3.12413907051</min_angle>
+            <max_angle>3.12413907051</max_angle>
+          </horizontal>
+        </scan>
+        <range>
+          <min>0.15</min>
+          <max>12</max>
+          <resolution>0.01</resolution>
+        </range>
+      </ray>
+      <plugin name="laser" filename="libRayPlugin.so" />
+      <plugin name="gazebo_ros_hokuyo_controller" filename="libgazebo_ros_laser.so">
+        <robotNamespace>$(arg prefix)</robotNamespace>
+        <topicName>scan</topicName>
+        <frameName>base_laser</frameName>
+      </plugin>
+      <always_on>1</always_on>
+      <update_rate>10</update_rate>
+      <visualize>true</visualize>
+    </sensor>
   </gazebo>
   <gazebo reference="$(arg prefix)/kinect_ros_link">
     <sensor name="camera" type="depth">
-        <update_rate>20</update_rate>
-        <camera>
-          <horizontal_fov>1.047198</horizontal_fov>
-          <image>
-            <width>640</width>
-            <height>480</height>
-            <format>R8G8B8</format>
-          </image>
-          <clip>
-            <near>0.05</near>
-            <far>3</far>
-          </clip>
-        </camera>
-        <plugin name="camera_plugin" filename="libgazebo_ros_openni_kinect.so">
-          <robotNamespace>$(arg prefix)</robotNamespace>
-          <baseline>0.2</baseline>
-          <alwaysOn>true</alwaysOn>
-          <!-- Keep this zero, update_rate in the parent <sensor> tag
-            will control the frame rate. -->
-          <updateRate>0.0</updateRate>
-          <cameraName>camera_ir</cameraName>
-          <!--imageTopicName>/camera/color/image_raw</imageTopicName>
-          <cameraInfoTopicName>/camera/color/camera_info</cameraInfoTopicName>
-          <depthImageTopicName>/camera/depth/image_raw</depthImageTopicName>
-          <depthImageCameraInfoTopicName>/camera/depth/camera_info</depthImageCameraInfoTopicName>
-          <pointCloudTopicName>/camera/depth/points</pointCloudTopicName-->
-          <frameName>camera_link</frameName>
-          <pointCloudCutoff>0.5</pointCloudCutoff>
-          <pointCloudCutoffMax>3.0</pointCloudCutoffMax>
-          <distortionK1>0</distortionK1>
-          <distortionK2>0</distortionK2>
-          <distortionK3>0</distortionK3>
-          <distortionT1>0</distortionT1>
-          <distortionT2>0</distortionT2>
-          <CxPrime>0</CxPrime>
-          <Cx>0</Cx>
-          <Cy>0</Cy>
-          <focalLength>0</focalLength>
-          <hackBaseline>0</hackBaseline>
-        </plugin>
-      </sensor>
+      <update_rate>20</update_rate>
+      <camera>
+        <horizontal_fov>1.047198</horizontal_fov>
+        <image>
+          <width>640</width>
+          <height>480</height>
+          <format>R8G8B8</format>
+        </image>
+        <clip>
+          <near>0.05</near>
+          <far>3</far>
+        </clip>
+      </camera>
+      <plugin name="camera_plugin" filename="libgazebo_ros_openni_kinect.so">
+        <robotNamespace>$(arg prefix)</robotNamespace>
+        <baseline>0.2</baseline>
+        <alwaysOn>true</alwaysOn>
+        <!-- Keep this zero, update_rate in the parent <sensor> tag
+ will control the frame rate. -->
+        <updateRate>0.0</updateRate>
+        <cameraName>camera_ir</cameraName>
+        <!--imageTopicName>/camera/color/image_raw</imageTopicName>
+ <cameraInfoTopicName>/camera/color/camera_info</cameraInfoTopicName>
+ <depthImageTopicName>/camera/depth/image_raw</depthImageTopicName>
+ <depthImageCameraInfoTopicName>/camera/depth/camera_info</depthImageCameraInfoTopicName>
+ <pointCloudTopicName>/camera/depth/points</pointCloudTopicName-->
+        <frameName>camera_link</frameName>
+        <pointCloudCutoff>0.5</pointCloudCutoff>
+        <pointCloudCutoffMax>3.0</pointCloudCutoffMax>
+        <distortionK1>0</distortionK1>
+        <distortionK2>0</distortionK2>
+        <distortionK3>0</distortionK3>
+        <distortionT1>0</distortionT1>
+        <distortionT2>0</distortionT2>
+        <CxPrime>0</CxPrime>
+        <Cx>0</Cx>
+        <Cy>0</Cy>
+        <focalLength>0</focalLength>
+        <hackBaseline>0</hackBaseline>
+      </plugin>
+    </sensor>
   </gazebo>
   <gazebo reference="$(arg prefix)/imu_link">
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