Commit message: pioneers config and launch files changes (#4)
* Removed movement limitation / set to speed control

Controller can now be controlled by settings up their velocity thorugh the controller command.

* Necessary config for controllers

* Controllers config changes

* Add dependancies catkin_EXPORTED_TARGETS to tf_publisher, interCommunication and communicationBroker to make sure that .msg are build before the applications

* Fixed the odometry publishing. Remove the joint_state_controller transmission because the odometry plugin has a built differential controller easier to use. Changed the child link of the tf_publisher for /odom since the odomertry plugin publish a tf between /odom and base_footprint

* Changed the directory of the meshes to be more close to root. Deleted the models directory since it's now useless

* Remove launchfile from swarmus_ros_description

* Auto stash before merge of "SWARINFO-47_create-high-level-hiveboard" and "origin/SWARINFO-47_create-high-level-hiveboard"

Only use pioneer_spawner launch file when adding pioneer

* Spawning pioneers from launch file

* Changed castor for caster in the URDF

* Fix PR

PR: https://github.com/SwarmUS/SwarmUS-ROS/pull/4

Co-authored-by: e-vil <etienne.villemure@usherbrooke.ca>

File: swarmus_ros_description/urdf/pioneer.urdf.xacro (robot description, xacro)
@@ -27,5 +27,5 @@
       <origin rpy="0 0 0" xyz="0 0 0.04"/>
       <geometry>
-        <mesh filename="package://swarmus_ros_description/models/pioneer_swarmus/meshes/chassis.dae" scale="1.0 1.0 1.0"/>
+        <mesh filename="package://swarmus_ros_description/meshes/chassis.dae" scale="1.0 1.0 1.0"/>
       </geometry>
     </visual>
@@ -103,5 +103,5 @@
       <origin rpy="0 0 0" xyz="0 0 0.03599"/>
       <geometry>
-        <mesh filename="package://swarmus_ros_description/models/kinect_ros/meshes/kinect.dae" scale="1.0 1.0 1.0"/>
+        <mesh filename="package://swarmus_ros_description/meshes/kinect.dae" scale="1.0 1.0 1.0"/>
       </geometry>
     </visual>
@@ -127,5 +127,5 @@
     <visual name="visual">
       <geometry>
-        <mesh filename="package://swarmus_ros_description/models/rplidar/meshes/hokuyo.dae" scale="1.0 1.0 1.0"/>
+        <mesh filename="package://swarmus_ros_description/meshes/hokuyo.dae" scale="1.0 1.0 1.0"/>
       </geometry>
     </visual>
@@ -163,6 +163,5 @@
     <origin rpy="0 1.5707 1.5707" xyz="0.1 0.17 -0.05"/>
     <axis xyz="9.00000000e-05 9.00000000e-05 1.00000000e+00"/>
-    <limit effort="0.0" velocity="0.0"/>
->
+    <limit effort="100.0" velocity="100"/>
   </joint>
   <joint name="right_wheel_hinge" type="continuous">
@@ -171,5 +170,5 @@
     <origin rpy="0 1.5707 1.5707" xyz="0.1 -0.17 -0.05"/>
     <axis xyz="9.00000000e-05 9.00000000e-05 1.00000000e+00"/>
-    <limit effort="0.0" velocity="0.0"/>
+    <limit effort="100.0" velocity="100"/>
   </joint>
   <joint name="imu_joint" type="fixed">
@@ -218,11 +217,8 @@
   </gazebo>
   <gazebo>
-    <plugin name="gazebo_ros_control" filename="libgazebo_ros_control.so">
-      <robotSimType>gazebo_ros_control/DefaultRobotHWSim</robotSimType>
-    </plugin>
+    <plugin name="gazebo_ros_control" filename="libgazebo_ros_control.so"/>
   </gazebo>
   <gazebo>
     <plugin name="differential_drive" filename="libgazebo_ros_diff_drive.so">
-      <robotNamespace>$(arg prefix)</robotNamespace>
       <commandTopic>cmd_vel</commandTopic>
       <odometryTopic>odom</odometryTopic>
@@ -230,5 +226,5 @@
       <odometrySource>world</odometrySource>
       <publishOdomTF>true</publishOdomTF>
-      <robotBaseFrame>$(arg prefix)/base_footprint</robotBaseFrame>
+      <robotBaseFrame>base_footprint</robotBaseFrame>
       <publishWheelTF>false</publishWheelTF>
       <publishTf>true</publishTf>
@@ -236,42 +232,42 @@
       <legacyMode>false</legacyMode>
       <updateRate>50</updateRate>
-      <leftJoint>$(arg prefix)/left_wheel</leftJoint>
-      <rightJoint>$(arg prefix)/right_wheel</rightJoint>
+      <leftJoint>left_wheel_hinge</leftJoint>
+      <rightJoint>right_wheel_hinge</rightJoint>
       <wheelSeparation>0.34</wheelSeparation>
       <wheelDiameter>0.22</wheelDiameter>
       <wheelAcceleration>1</wheelAcceleration>
       <wheelTorque>10</wheelTorque>
-      <rosDebugLevel>na</rosDebugLevel>
+      <rosDebugLevel>true</rosDebugLevel>
     </plugin>
   </gazebo>
   <gazebo reference="$(arg prefix)/rplidar">
-    <sensor name="laser" type="ray">
-      <pose>0.01 0 0.0175 0 -0 0</pose>
-      <ray>
-        <scan>
-          <horizontal>
-            <!-- Specs from racecar's rplidar -->base_lidar
-            <samples>360</samples>
-            <resolution>1</resolution>
-            <min_angle>-3.12413907051</min_angle>
-            <max_angle>3.12413907051</max_angle>
-          </horizontal>
-        </scan>
-        <range>
-          <min>0.15</min>
-          <max>12</max>
-          <resolution>0.01</resolution>
-        </range>
-      </ray>
-      <plugin name="laser" filename="libRayPlugin.so" />
-      <plugin name="gazebo_ros_hokuyo_controller" filename="libgazebo_ros_laser.so">
-        <robotNamespace>$(arg prefix)</robotNamespace>
-        <topicName>scan</topicName>
-        <frameName>base_laser</frameName>
-      </plugin>
-      <always_on>1</always_on>
-      <update_rate>10</update_rate>
-      <visualize>true</visualize>
-    </sensor>
+      <sensor name="laser" type="ray">
+        <pose>0.01 0 0.0175 0 -0 0</pose>
+        <ray>
+          <scan>
+            <horizontal>
+              <!-- Specs from racecar's rplidar -->base_lidar
+              <samples>360</samples>
+              <resolution>1</resolution>
+              <min_angle>-3.12413907051</min_angle>
+              <max_angle>3.12413907051</max_angle>
+            </horizontal>
+          </scan>
+          <range>
+            <min>0.15</min>
+            <max>12</max>
+            <resolution>0.01</resolution>
+          </range>
+        </ray>
+        <plugin name="laser" filename="libRayPlugin.so" />
+        <plugin name="gazebo_ros_hokuyo_controller" filename="libgazebo_ros_laser.so">
+          <robotNamespace>$(arg prefix)</robotNamespace>
+          <topicName>scan</topicName>
+          <frameName>base_laser</frameName>
+        </plugin>
+        <always_on>1</always_on>
+        <update_rate>10</update_rate>
+        <visualize>false</visualize>
+      </sensor>
   </gazebo>
   <gazebo reference="$(arg prefix)/kinect_ros_link">
@@ -333,22 +329,3 @@
     </sensor>
   </gazebo>
-  <!-- ================================== Transmission ================================== -->
-  <transmission name="$(arg prefix)_right_wheel_trans">
-    <type>transmission_interface/SimpleTransmission</type>
-    <actuator name="$(arg prefix)_right_wheel_motor">
-      <mechanicalReduction>1</mechanicalReduction>
-    </actuator>
-    <joint name="right_wheel_hinge">
-      <hardwareInterface>hardware_interface/EffortJointInterface</hardwareInterface>
-    </joint>
-  </transmission>
-  <transmission name="$(arg prefix)_left_wheel_trans">
-    <type>transmission_interface/SimpleTransmission</type>
-    <actuator name="$(arg prefix)_left_wheel_motor">
-      <mechanicalReduction>1</mechanicalReduction>
-    </actuator>
-    <joint name="left_wheel_hinge">
-      <hardwareInterface>hardware_interface/EffortJointInterface</hardwareInterface>
-    </joint>
-  </transmission>
 </robot>

Commit message: Kinect fixes
-Added kinect to RVIZ configuration
-Changed pioneer_0's default orientation
-Changed pointcloud orientation

File: swarmus_ros_description/urdf/pioneer.urdf.xacro (robot description, xacro)
@@ -107,4 +107,6 @@
     </visual>
   </link>
+  <link name="$(arg prefix)/kinect_optical_ros_link">
+  </link>
   <link name="$(arg prefix)/rplidar">
     <inertial>
@@ -183,4 +185,9 @@
     <parent link="$(arg prefix)/chassis" />
     <origin rpy="0 0 0" xyz="0.20 0 0.11"/>
+  </joint>
+  <joint name="kinect_optical_joint" type="fixed">
+    <origin xyz="0 0 0" rpy="${-pi/2} 0 ${-pi/2}"/>
+    <parent link="$(arg prefix)/kinect_ros_link"/>
+    <child link="$(arg prefix)/kinect_optical_ros_link"/>
   </joint>
   <joint name="rplidar_joint" type="fixed">
@@ -299,5 +306,5 @@
  <depthImageCameraInfoTopicName>/camera/depth/camera_info</depthImageCameraInfoTopicName>
  <pointCloudTopicName>/camera/depth/points</pointCloudTopicName-->
-        <frameName>kinect_ros_link</frameName>
+        <frameName>kinect_optical_ros_link</frameName>
         <pointCloudCutoff>0.5</pointCloudCutoff>
         <pointCloudCutoffMax>3.0</pointCloudCutoffMax>

Commit message: Added kinect texture to Gazebo

File: swarmus_ros_description/urdf/pioneer.urdf.xacro (robot description, xacro)
@@ -3,4 +3,5 @@
   xmlns:xacro="http://www.ros.org/wiki/xacro">
   <xacro:arg name="prefix" default="p_swarmus"/>
+  <xacro:arg name="color" default="DepthMapVS"/>
   <link name="$(arg prefix)/base_footprint" />
   <link name="$(arg prefix)/base_link" />
@@ -321,4 +322,5 @@
       </plugin>
     </sensor>
+    <material>Gazebo/$(arg color)</material>
   </gazebo>
   <gazebo reference="$(arg prefix)/imu_link">
