Commit message: Moved the Pioneer's base_footprint
- Moved the base_footprint in the Pioneer's URDF to the barycenter of the motors (between the motors) instead of being below the robot's center.  This is needed to have a proper differential drive controller.

File: src/swarmus_ros_description/urdf/pioneer.urdf.xacro (robot description, xacro)
@@ -152,5 +152,5 @@
   <!-- ================================== Joints ==================================-->
   <joint name="base_footprint_link_joint" type="fixed">
-    <origin xyz="0 0 0.16" rpy="0 0 0" />
+    <origin xyz="-0.1 0 0.16" rpy="0 0 0" />
     <parent link="$(arg prefix)/base_footprint" />
     <child link="$(arg prefix)/base_link" />

Commit message: Changed the camera position and orientation in URDF
- Those are the real position and orientation on the robot

File: src/swarmus_ros_description/urdf/pioneer.urdf.xacro (robot description, xacro)
@@ -185,5 +185,5 @@
     <child link="$(arg prefix)/kinect_ros_link" />
     <parent link="$(arg prefix)/chassis" />
-    <origin rpy="0 0 0" xyz="0.20 0 0.11"/>
+    <origin rpy="0 -0.174553 0" xyz="0.18059 0 0.16048"/>
   </joint>
   <joint name="kinect_optical_joint" type="fixed">

Commit message: URDF Update
- Changed the rplidar positions to have a similar position to the lidar placement of the real robot
- Removed the collision box of the Kinect since it was blocking the lidar.

File: src/swarmus_ros_description/urdf/pioneer.urdf.xacro (robot description, xacro)
@@ -95,10 +95,4 @@
       <inertia ixx="0" ixy="0" ixz="0" iyy="0" iyz="0" izz="0"/>
     </inertial>
-    <collision name="collision">
-      <origin rpy="0 0 0" xyz="0 0 0.03599"/>
-      <geometry>
-        <box size="0.073000 0.276000 0.072000"/>
-      </geometry>
-    </collision>
     <visual name="visual">
       <origin rpy="0 0 0" xyz="0 0 0.03599"/>
@@ -195,5 +189,5 @@
     <child link="$(arg prefix)/rplidar"/>
     <parent link="$(arg prefix)/chassis" />
-    <origin rpy="0 0 0" xyz="0 0 0.21"/>
+    <origin rpy="0 0 0" xyz="0.02378 0 0.19709"/>
   </joint>
   <joint name="hiveboard_joint" type="fixed">

Commit message: Added simulated realsense
- Added condition to set the simulated camera to the d435i or the d455
- Changed the resolution to match the depth sensor resolution of the d435i and the d455. It should be noted that the RGB resolution of the d455 is slightly different and the RGB resolution is greatly different compared to their depth resolution. Since only there is only one resolution parameter, I took the depth one.
- Changed the cutoff distance of the point cloud and the depth sensor to the manufacturer specifications
- Set the default camera for the simulated pioneer to the d435i

File: src/swarmus_ros_description/urdf/pioneer.urdf.xacro (robot description, xacro)
@@ -4,4 +4,6 @@
   <xacro:arg name="prefix" default="p_swarmus"/>
   <xacro:arg name="color" default="DepthMapVS"/>
+  <xacro:arg name="camera_type" default="d435i"/>
+  <xacro:property name="camera_type" value="$(arg camera_type)"/>
   <link name="$(arg prefix)/base_footprint" />
   <link name="$(arg prefix)/base_link" />
@@ -275,11 +277,16 @@
   <gazebo reference="$(arg prefix)/kinect_ros_link">
     <sensor name="camera" type="depth">
-      <update_rate>20</update_rate>
+      <update_rate>30</update_rate>
       <camera>
-        <horizontal_fov>1.047198</horizontal_fov>
+        <xacro:if value="${camera_type == 'd435i'}">
+          <horizontal_fov>1.117</horizontal_fov> <!-- 64 deg field of view of the RGDB sensor used since its smaller than the depth FOV-->
+        </xacro:if>
+        <xacro:if value="${camera_type == 'd455'}">
+          <horizontal_fov>1.501</horizontal_fov> <!-- 86 deg field of view of the depth sensor used- since its smaller than the RGBD value-->
+        </xacro:if>
         <image>
-          <width>640</width>
-          <height>480</height>
-          <format>R8G8B8</format>
+            <width>1280</width>
+            <height>720</height>
+            <format>R8G8B8</format>
         </image>
         <clip>
@@ -293,15 +300,21 @@
         <alwaysOn>true</alwaysOn>
         <!-- Keep this zero, update_rate in the parent <sensor> tag
- will control the frame rate. -->
+will control the frame rate. -->
         <updateRate>0.0</updateRate>
         <cameraName>camera_ir</cameraName>
         <!--imageTopicName>/camera/color/image_raw</imageTopicName>
- <cameraInfoTopicName>/camera/color/camera_info</cameraInfoTopicName>
- <depthImageTopicName>/camera/depth/image_raw</depthImageTopicName>
- <depthImageCameraInfoTopicName>/camera/depth/camera_info</depthImageCameraInfoTopicName>
- <pointCloudTopicName>/camera/depth/points</pointCloudTopicName-->
+<cameraInfoTopicName>/camera/color/camera_info</cameraInfoTopicName>
+<depthImageTopicName>/camera/depth/image_raw</depthImageTopicName>
+<depthImageCameraInfoTopicName>/camera/depth/camera_info</depthImageCameraInfoTopicName>
+<pointCloudTopicName>/camera/depth/points</pointCloudTopicName-->
+        <xacro:if value="${camera_type == 'd435i'}">
+          <pointCloudCutoff>0.3</pointCloudCutoff>
+          <pointCloudCutoffMax>3</pointCloudCutoffMax>
+        </xacro:if>
+        <xacro:if value="${camera_type == 'd455'}">
+          <pointCloudCutoff>0.6</pointCloudCutoff>
+          <pointCloudCutoffMax>6</pointCloudCutoffMax>
+        </xacro:if>
         <frameName>kinect_optical_ros_link</frameName>
-        <pointCloudCutoff>1.2</pointCloudCutoff>
-        <pointCloudCutoffMax>3.5</pointCloudCutoffMax>
         <distortionK1>0</distortionK1>
         <distortionK2>0</distortionK2>

Commit message: Moved the simulated IMU on the camera
- Removed the IMU link since it will used the camera link
- Changed the IMU parameters since the values were not relevant

File: src/swarmus_ros_description/urdf/pioneer.urdf.xacro (robot description, xacro)
@@ -78,17 +78,4 @@
     </visual>
   </link>
-  <link name="$(arg prefix)/imu_link">
-    <inertial>
-      <mass value="0.0000001"/>
-      <origin rpy="0 0 0" xyz="0 0 0"/>
-      <inertia ixx="0.00001" ixy="0" ixz="0" iyy="0.00001" iyz="0" izz="0.00001"/>
-    </inertial>
-    <visual name="pioneer_swarmus__visual">
-      <origin rpy="0 0 0" xyz="0 0 0"/>
-      <geometry>
-        <box size="0.03 0.03 0.01"/>
-      </geometry>
-    </visual>
-  </link>
   <link name="$(arg prefix)/kinect_ros_link">
     <inertial>
@@ -170,11 +157,4 @@
     <axis xyz="9.00000000e-05 9.00000000e-05 1.00000000e+00"/>
     <limit effort="100.0" velocity="100"/>
-  </joint>
-  <joint name="imu_joint" type="fixed">
-    <parent link="$(arg prefix)/chassis"/>
-    <child link="$(arg prefix)/imu_link"/>
-    <origin rpy="0 0 0" xyz="0.07 0 0.11"/>
-    <axis xyz="0 0 0"/>
-    <limit effort="0" velocity="0"/>
   </joint>
   <joint name="kinect_joint" type="fixed">
@@ -331,15 +311,19 @@
     <material>Gazebo/$(arg color)</material>
   </gazebo>
-  <gazebo reference="$(arg prefix)/imu_link">
+  <gazebo reference="$(arg prefix)/kinect_optical_ros_link">
+    <gravity>true</gravity>
     <sensor name="imu_sensor" type="imu">
+      <alwaysOn>true</alwaysOn>
+      <update_rate>100</update_rate>
       <plugin filename="libgazebo_ros_imu_sensor.so" name="imu_plugin">
         <robotNamespace>$(arg prefix)</robotNamespace>
-        <topicName>imu/data</topicName>
-        <bodyName>$(arg prefix)/imu_link</bodyName>
+        <topicName>camera/imu</topicName>
+        <bodyName>$(arg prefix)/kinect_optical_ros_link</bodyName>
         <updateRateHZ>100</updateRateHZ>
-        <gaussianNoise>0.01</gaussianNoise>
+        <gaussianNoise>0.0</gaussianNoise>
         <xyzOffset>0 0 0</xyzOffset>
         <rpyOffset>0 0 0</rpyOffset>
-        <frameName>$(arg prefix)/imu_link</frameName>
+        <frameName>$(arg prefix)/kinect_optical_ros_link</frameName>
+        <initialOrientationAsReference>false</initialOrientationAsReference>
       </plugin>
     </sensor>

Commit message: Replaced Kinect with realsense_description
- Removed the Kinect frame and include the realsense2_description package to include the D435i modal. 
- Remaped the simulated snesors to the realsense frame
- Added a  runtime dependency to the realsense2_description package

File: src/swarmus_ros_description/urdf/pioneer.urdf.xacro (robot description, xacro)
@@ -2,8 +2,10 @@
 <robot name="pioneer_swarmus"
   xmlns:xacro="http://www.ros.org/wiki/xacro">
+  <xacro:include filename="$(find realsense2_description)/urdf/_d435i.urdf.xacro"/>
   <xacro:arg name="prefix" default="p_swarmus"/>
   <xacro:arg name="color" default="DepthMapVS"/>
   <xacro:arg name="camera_type" default="d435i"/>
   <xacro:property name="camera_type" value="$(arg camera_type)"/>
+  <xacro:arg name="use_nominal_extrinsics" default="true" />
   <link name="$(arg prefix)/base_footprint" />
   <link name="$(arg prefix)/base_link" />
@@ -78,19 +80,7 @@
     </visual>
   </link>
-  <link name="$(arg prefix)/kinect_ros_link">
-    <inertial>
-      <mass value="0.1"/>
-      <origin rpy="0 0 0" xyz="0 0 0"/>
-      <inertia ixx="0" ixy="0" ixz="0" iyy="0" iyz="0" izz="0"/>
-    </inertial>
-    <visual name="visual">
-      <origin rpy="0 0 0" xyz="0 0 0.03599"/>
-      <geometry>
-        <mesh filename="package://swarmus_ros_description/meshes/kinect.dae" scale="1.0 1.0 1.0"/>
-      </geometry>
-    </visual>
-  </link>
-  <link name="$(arg prefix)/kinect_optical_ros_link">
-  </link>
+  <xacro:sensor_d435i parent="$(arg prefix)/chassis" name="$(arg prefix)/camera" use_nominal_extrinsics="$(arg use_nominal_extrinsics)">
+    <origin xyz="0.16773 0 0.14602" rpy="0 -0.174553 0"/>
+  </xacro:sensor_d435i>
   <link name="$(arg prefix)/rplidar">
     <inertial>
@@ -157,14 +147,4 @@
     <axis xyz="9.00000000e-05 9.00000000e-05 1.00000000e+00"/>
     <limit effort="100.0" velocity="100"/>
-  </joint>
-  <joint name="kinect_joint" type="fixed">
-    <child link="$(arg prefix)/kinect_ros_link" />
-    <parent link="$(arg prefix)/chassis" />
-    <origin rpy="0 -0.174553 0" xyz="0.18059 0 0.16048"/>
-  </joint>
-  <joint name="kinect_optical_joint" type="fixed">
-    <origin xyz="0 0 0" rpy="${-pi/2} 0 ${-pi/2}"/>
-    <parent link="$(arg prefix)/kinect_ros_link"/>
-    <child link="$(arg prefix)/kinect_optical_ros_link"/>
   </joint>
   <joint name="rplidar_joint" type="fixed">
@@ -255,5 +235,5 @@
       </sensor>
   </gazebo>
-  <gazebo reference="$(arg prefix)/kinect_ros_link">
+  <gazebo reference="$(arg prefix)/camera_depth_frame">
     <sensor name="camera" type="depth">
       <update_rate>30</update_rate>
@@ -282,5 +262,5 @@
 will control the frame rate. -->
         <updateRate>0.0</updateRate>
-        <cameraName>camera_ir</cameraName>
+        <cameraName>camera</cameraName>
         <!--imageTopicName>/camera/color/image_raw</imageTopicName>
 <cameraInfoTopicName>/camera/color/camera_info</cameraInfoTopicName>
@@ -296,5 +276,5 @@
           <pointCloudCutoffMax>6</pointCloudCutoffMax>
         </xacro:if>
-        <frameName>kinect_optical_ros_link</frameName>
+        <frameName>camera_depth_optical_frame</frameName>
         <distortionK1>0</distortionK1>
         <distortionK2>0</distortionK2>
@@ -311,5 +291,5 @@
     <material>Gazebo/$(arg color)</material>
   </gazebo>
-  <gazebo reference="$(arg prefix)/kinect_optical_ros_link">
+  <gazebo reference="$(arg prefix)/camera_accel_optical_frame">
     <gravity>true</gravity>
     <sensor name="imu_sensor" type="imu">
@@ -319,10 +299,10 @@
         <robotNamespace>$(arg prefix)</robotNamespace>
         <topicName>camera/imu</topicName>
-        <bodyName>$(arg prefix)/kinect_optical_ros_link</bodyName>
+        <bodyName>$(arg prefix)/camera_accel_optical_frame</bodyName>
         <updateRateHZ>100</updateRateHZ>
         <gaussianNoise>0.0</gaussianNoise>
         <xyzOffset>0 0 0</xyzOffset>
         <rpyOffset>0 0 0</rpyOffset>
-        <frameName>$(arg prefix)/kinect_optical_ros_link</frameName>
+        <frameName>$(arg prefix)/camera_accel_optical_frame</frameName>
         <initialOrientationAsReference>false</initialOrientationAsReference>
       </plugin>

Commit message: Added the D455 to Pioneer
- Added the D455 URDF to the pioneer URDF
- Changed the name of  topics to match the realsense topics

File: src/swarmus_ros_description/urdf/pioneer.urdf.xacro (robot description, xacro)
@@ -2,5 +2,4 @@
 <robot name="pioneer_swarmus"
   xmlns:xacro="http://www.ros.org/wiki/xacro">
-  <xacro:include filename="$(find realsense2_description)/urdf/_d435i.urdf.xacro"/>
   <xacro:arg name="prefix" default="p_swarmus"/>
   <xacro:arg name="color" default="DepthMapVS"/>
@@ -80,7 +79,16 @@
     </visual>
   </link>
-  <xacro:sensor_d435i parent="$(arg prefix)/chassis" name="$(arg prefix)/camera" use_nominal_extrinsics="$(arg use_nominal_extrinsics)">
-    <origin xyz="0.16773 0 0.14602" rpy="0 -0.174553 0"/>
-  </xacro:sensor_d435i>
+  <xacro:if value="${camera_type == 'd435i'}">
+    <xacro:include filename="$(find realsense2_description)/urdf/_d435i.urdf.xacro"/>
+    <xacro:sensor_d435i parent="$(arg prefix)/chassis" name="$(arg prefix)/camera" use_nominal_extrinsics="$(arg use_nominal_extrinsics)">
+      <origin xyz="0.16773 0 0.14602" rpy="0 -0.174553 0"/>
+    </xacro:sensor_d435i>
+  </xacro:if>
+  <xacro:if value="${camera_type == 'd455'}">
+    <xacro:include filename="$(find realsense2_description)/urdf/_d455.urdf.xacro"/>
+    <xacro:sensor_d455 parent="$(arg prefix)/chassis" name="$(arg prefix)/camera" use_nominal_extrinsics="$(arg use_nominal_extrinsics)">
+      <origin xyz="0.16773 0 0.14602" rpy="0 -0.174553 0"/>
+    </xacro:sensor_d455>
+  </xacro:if>
   <link name="$(arg prefix)/rplidar">
     <inertial>
@@ -263,9 +271,9 @@
         <updateRate>0.0</updateRate>
         <cameraName>camera</cameraName>
-        <!--imageTopicName>/camera/color/image_raw</imageTopicName>
-<cameraInfoTopicName>/camera/color/camera_info</cameraInfoTopicName>
-<depthImageTopicName>/camera/depth/image_raw</depthImageTopicName>
-<depthImageCameraInfoTopicName>/camera/depth/camera_info</depthImageCameraInfoTopicName>
-<pointCloudTopicName>/camera/depth/points</pointCloudTopicName-->
+        <imageTopicName>color/image_raw</imageTopicName>
+        <cameraInfoTopicName>color/camera_info</cameraInfoTopicName>
+        <depthImageTopicName>depth/image_rect_raw</depthImageTopicName>
+        <depthImageCameraInfoTopicName>depth/camera_info</depthImageCameraInfoTopicName>
+        <pointCloudTopicName>depth/color/points</pointCloudTopicName>
         <xacro:if value="${camera_type == 'd435i'}">
           <pointCloudCutoff>0.3</pointCloudCutoff>
