Commit message: Feat/swarinfo 120 urdf update (#23)
* Updated dependencies

- Changed the rosdep2 for the packages suggested by the ROS noetic installation guide

* Changed the camera position and orientation in URDF

- Those are the real position and orientation on the robot

* URDF Update

- Changed the rplidar positions to have a similar position to the lidar placement of the real robot
- Removed the collision box of the Kinect since it was blocking the lidar.

* Added simulated realsense

- Added condition to set the simulated camera to the d435i or the d455
- Changed the resolution to match the depth sensor resolution of the d435i and the d455. It should be noted that the RGB resolution of the d455 is slightly different and the RGB resolution is greatly different compared to their depth resolution. Since only there is only one resolution parameter, I took the depth one.
- Changed the cutoff distance of the point cloud and the depth sensor to the manufacturer specifications
- Set the default camera for the simulated pioneer to the d435i

* Moved the simulated IMU on the camera

- Removed the IMU link since it will used the camera link
- Changed the IMU parameters since the values were not relevant

* Replaced Kinect with realsense_description

- Removed the Kinect frame and include the realsense2_description package to include the D435i modal. 
- Remaped the simulated snesors to the realsense frame
- Added a  runtime dependency to the realsense2_description package

* Removed realsense submodule

* Added forked Realsense-ROS

-Added a forked version of Realsense-ROS that contains the d455 URDF

* Switched submodule branch

- Changed branch where the D455 URDFs are defined

* WIP

* Added forked realsense-ros

- Added a fork of the realsense-ros repo that contains URDF and materials for the D455

* Checkout d455 branch

* Remove old realsense-ros module

* Added the D455 to Pioneer

- Added the D455 URDF to the pioneer URDF
- Changed the name of  topics to match the realsense topics

* Updated RVIZ

-Changed the topics of the camera modules (kinect and pointcloud) to work with the latest topic naming.

* Added simulation flag

- Added an argument that can be set to load the gazebo plugins and to publish the nominal TFs of the camera

* Changed RTAB-map subscribed topics  

- Changed topic names to match the new ones

* Adjusted position of D455

-Adjusted the D455 origin since the distance in x between the screw mount and the depth frame is not the same for the D455 and the D435i

Co-authored-by: Etienne <vile2094@usherbrooke.ca>

File: src/swarmus_ros_description/urdf/pioneer.urdf.xacro (robot description, xacro)
@@ -4,4 +4,8 @@
   <xacro:arg name="prefix" default="p_swarmus"/>
   <xacro:arg name="color" default="DepthMapVS"/>
+  <xacro:arg name="camera_type" default="d435i"/>
+  <xacro:property name="camera_type" value="$(arg camera_type)"/>
+  <xacro:arg name="is_simulation" default="false"/>
+  <xacro:property name="is_simulation" value="$(arg is_simulation)"/>
   <link name="$(arg prefix)/base_footprint" />
   <link name="$(arg prefix)/base_link" />
@@ -76,38 +80,16 @@
     </visual>
   </link>
-  <link name="$(arg prefix)/imu_link">
-    <inertial>
-      <mass value="0.0000001"/>
-      <origin rpy="0 0 0" xyz="0 0 0"/>
-      <inertia ixx="0.00001" ixy="0" ixz="0" iyy="0.00001" iyz="0" izz="0.00001"/>
-    </inertial>
-    <visual name="pioneer_swarmus__visual">
-      <origin rpy="0 0 0" xyz="0 0 0"/>
-      <geometry>
-        <box size="0.03 0.03 0.01"/>
-      </geometry>
-    </visual>
-  </link>
-  <link name="$(arg prefix)/kinect_ros_link">
-    <inertial>
-      <mass value="0.1"/>
-      <origin rpy="0 0 0" xyz="0 0 0"/>
-      <inertia ixx="0" ixy="0" ixz="0" iyy="0" iyz="0" izz="0"/>
-    </inertial>
-    <collision name="collision">
-      <origin rpy="0 0 0" xyz="0 0 0.03599"/>
-      <geometry>
-        <box size="0.073000 0.276000 0.072000"/>
-      </geometry>
-    </collision>
-    <visual name="visual">
-      <origin rpy="0 0 0" xyz="0 0 0.03599"/>
-      <geometry>
-        <mesh filename="package://swarmus_ros_description/meshes/kinect.dae" scale="1.0 1.0 1.0"/>
-      </geometry>
-    </visual>
-  </link>
-  <link name="$(arg prefix)/kinect_optical_ros_link">
-  </link>
+  <xacro:if value="${camera_type == 'd435i'}">
+    <xacro:include filename="$(find realsense2_description)/urdf/_d435i.urdf.xacro"/>
+    <xacro:sensor_d435i parent="$(arg prefix)/chassis" name="$(arg prefix)/camera" use_nominal_extrinsics="${is_simulation}">
+      <origin xyz="0.16773 0 0.14602" rpy="0 -0.174553 0"/>
+    </xacro:sensor_d435i>
+  </xacro:if>
+  <xacro:if value="${camera_type == 'd455'}">
+    <xacro:include filename="$(find realsense2_description)/urdf/_d455.urdf.xacro"/>
+    <xacro:sensor_d455 parent="$(arg prefix)/chassis" name="$(arg prefix)/camera" use_nominal_extrinsics="${is_simulation}">
+      <origin xyz="0.16822 0 0.14357" rpy="0 -0.174553 0"/>
+    </xacro:sensor_d455>
+  </xacro:if>
   <link name="$(arg prefix)/rplidar">
     <inertial>
@@ -175,25 +157,8 @@
     <limit effort="100.0" velocity="100"/>
   </joint>
-  <joint name="imu_joint" type="fixed">
-    <parent link="$(arg prefix)/chassis"/>
-    <child link="$(arg prefix)/imu_link"/>
-    <origin rpy="0 0 0" xyz="0.07 0 0.11"/>
-    <axis xyz="0 0 0"/>
-    <limit effort="0" velocity="0"/>
-  </joint>
-  <joint name="kinect_joint" type="fixed">
-    <child link="$(arg prefix)/kinect_ros_link" />
-    <parent link="$(arg prefix)/chassis" />
-    <origin rpy="0 0 0" xyz="0.20 0 0.11"/>
-  </joint>
-  <joint name="kinect_optical_joint" type="fixed">
-    <origin xyz="0 0 0" rpy="${-pi/2} 0 ${-pi/2}"/>
-    <parent link="$(arg prefix)/kinect_ros_link"/>
-    <child link="$(arg prefix)/kinect_optical_ros_link"/>
-  </joint>
   <joint name="rplidar_joint" type="fixed">
     <child link="$(arg prefix)/rplidar"/>
     <parent link="$(arg prefix)/chassis" />
-    <origin rpy="0 0 0" xyz="0 0 0.21"/>
+    <origin rpy="0 0 0" xyz="0.02378 0 0.19709"/>
   </joint>
   <joint name="hiveboard_joint" type="fixed">
@@ -224,117 +189,133 @@
     <!-- material>Gazebo/$(arg color)</material-->
   </gazebo>
-  <gazebo>
-    <plugin name="gazebo_ros_control" filename="libgazebo_ros_control.so"/>
-  </gazebo>
-  <gazebo>
-    <plugin name="differential_drive" filename="libgazebo_ros_diff_drive.so">
-      <commandTopic>cmd_vel</commandTopic>
-      <odometryTopic>odom</odometryTopic>
-      <odometryFrame>odom</odometryFrame>
-      <odometrySource>world</odometrySource>
-      <publishOdomTF>true</publishOdomTF>
-      <robotBaseFrame>base_footprint</robotBaseFrame>
-      <publishWheelTF>false</publishWheelTF>
-      <publishTf>true</publishTf>
-      <publishWheelJointState>true</publishWheelJointState>
-      <legacyMode>false</legacyMode>
-      <updateRate>50</updateRate>
-      <leftJoint>left_wheel_hinge</leftJoint>
-      <rightJoint>right_wheel_hinge</rightJoint>
-      <wheelSeparation>0.34</wheelSeparation>
-      <wheelDiameter>0.22</wheelDiameter>
-      <wheelAcceleration>1</wheelAcceleration>
-      <wheelTorque>10</wheelTorque>
-      <rosDebugLevel>true</rosDebugLevel>
-    </plugin>
-  </gazebo>
-  <gazebo reference="$(arg prefix)/rplidar">
-      <sensor name="laser" type="ray">
-        <pose>0.01 0 0.0175 0 -0 0</pose>
-        <ray>
-          <scan>
-            <horizontal>
-              <!-- Specs from racecar's rplidar -->
-              <samples>360</samples>
-              <resolution>1</resolution>
-              <min_angle>-3.12413907051</min_angle>
-              <max_angle>3.12413907051</max_angle>
-            </horizontal>
-          </scan>
-          <range>
-            <min>0.15</min>
-            <max>12</max>
-            <resolution>0.01</resolution>
-          </range>
-        </ray>
-        <plugin name="laser" filename="libRayPlugin.so" />
-        <plugin name="gazebo_ros_hokuyo_controller" filename="libgazebo_ros_laser.so">
+  <xacro:if value="${is_simulation}">
+    <gazebo>
+      <plugin name="gazebo_ros_control" filename="libgazebo_ros_control.so"/>
+    </gazebo>
+    <gazebo>
+      <plugin name="differential_drive" filename="libgazebo_ros_diff_drive.so">
+        <commandTopic>cmd_vel</commandTopic>
+        <odometryTopic>odom</odometryTopic>
+        <odometryFrame>odom</odometryFrame>
+        <odometrySource>world</odometrySource>
+        <publishOdomTF>true</publishOdomTF>
+        <robotBaseFrame>base_footprint</robotBaseFrame>
+        <publishWheelTF>false</publishWheelTF>
+        <publishTf>true</publishTf>
+        <publishWheelJointState>true</publishWheelJointState>
+        <legacyMode>false</legacyMode>
+        <updateRate>50</updateRate>
+        <leftJoint>left_wheel_hinge</leftJoint>
+        <rightJoint>right_wheel_hinge</rightJoint>
+        <wheelSeparation>0.34</wheelSeparation>
+        <wheelDiameter>0.22</wheelDiameter>
+        <wheelAcceleration>1</wheelAcceleration>
+        <wheelTorque>10</wheelTorque>
+        <rosDebugLevel>true</rosDebugLevel>
+      </plugin>
+    </gazebo>
+    <gazebo reference="$(arg prefix)/rplidar">
+        <sensor name="laser" type="ray">
+          <pose>0.01 0 0.0175 0 -0 0</pose>
+          <ray>
+            <scan>
+              <horizontal>
+                <!-- Specs from racecar's rplidar -->
+                <samples>360</samples>
+                <resolution>1</resolution>
+                <min_angle>-3.12413907051</min_angle>
+                <max_angle>3.12413907051</max_angle>
+              </horizontal>
+            </scan>
+            <range>
+              <min>0.15</min>
+              <max>12</max>
+              <resolution>0.01</resolution>
+            </range>
+          </ray>
+          <plugin name="laser" filename="libRayPlugin.so" />
+          <plugin name="gazebo_ros_hokuyo_controller" filename="libgazebo_ros_laser.so">
+            <robotNamespace>$(arg prefix)</robotNamespace>
+            <topicName>scan</topicName>
+            <frameName>rplidar</frameName>
+          </plugin>
+          <always_on>1</always_on>
+          <update_rate>10</update_rate>
+          <visualize>false</visualize>
+        </sensor>
+    </gazebo>
+    <gazebo reference="$(arg prefix)/camera_depth_frame">
+      <sensor name="camera" type="depth">
+        <update_rate>30</update_rate>
+        <camera>
+          <xacro:if value="${camera_type == 'd435i'}">
+            <horizontal_fov>1.117</horizontal_fov> <!-- 64 deg field of view of the RGDB sensor used since its smaller than the depth FOV-->
+          </xacro:if>
+          <xacro:if value="${camera_type == 'd455'}">
+            <horizontal_fov>1.501</horizontal_fov> <!-- 86 deg field of view of the depth sensor used- since its smaller than the RGBD value-->
+          </xacro:if>
+          <image>
+              <width>1280</width>
+              <height>720</height>
+              <format>R8G8B8</format>
+          </image>
+          <clip>
+            <near>0.05</near>
+            <far>20</far>
+          </clip>
+        </camera>
+        <plugin name="camera_plugin" filename="libgazebo_ros_openni_kinect.so">
           <robotNamespace>$(arg prefix)</robotNamespace>
-          <topicName>scan</topicName>
-          <frameName>rplidar</frameName>
+          <baseline>0.2</baseline>
+          <alwaysOn>true</alwaysOn>
+          <!-- Keep this zero, update_rate in the parent <sensor> tag will control the frame rate. -->
+          <updateRate>0.0</updateRate>
+          <cameraName>camera</cameraName>
+          <imageTopicName>color/image_raw</imageTopicName>
+          <cameraInfoTopicName>color/camera_info</cameraInfoTopicName>
+          <depthImageTopicName>depth/image_rect_raw</depthImageTopicName>
+          <depthImageCameraInfoTopicName>depth/camera_info</depthImageCameraInfoTopicName>
+          <pointCloudTopicName>depth/color/points</pointCloudTopicName>
+          <xacro:if value="${camera_type == 'd435i'}">
+            <pointCloudCutoff>0.3</pointCloudCutoff>
+            <pointCloudCutoffMax>3</pointCloudCutoffMax>
+          </xacro:if>
+          <xacro:if value="${camera_type == 'd455'}">
+            <pointCloudCutoff>0.6</pointCloudCutoff>
+            <pointCloudCutoffMax>6</pointCloudCutoffMax>
+          </xacro:if>
+          <frameName>camera_depth_optical_frame</frameName>
+          <distortionK1>0</distortionK1>
+          <distortionK2>0</distortionK2>
+          <distortionK3>0</distortionK3>
+          <distortionT1>0</distortionT1>
+          <distortionT2>0</distortionT2>
+          <CxPrime>0</CxPrime>
+          <Cx>0</Cx>
+          <Cy>0</Cy>
+          <focalLength>0</focalLength>
+          <hackBaseline>0</hackBaseline>
         </plugin>
-        <always_on>1</always_on>
-        <update_rate>10</update_rate>
-        <visualize>false</visualize>
       </sensor>
-  </gazebo>
-  <gazebo reference="$(arg prefix)/kinect_ros_link">
-    <sensor name="camera" type="depth">
-      <update_rate>20</update_rate>
-      <camera>
-        <horizontal_fov>1.047198</horizontal_fov>
-        <image>
-          <width>640</width>
-          <height>480</height>
-          <format>R8G8B8</format>
-        </image>
-        <clip>
-          <near>0.05</near>
-          <far>20</far>
-        </clip>
-      </camera>
-      <plugin name="camera_plugin" filename="libgazebo_ros_openni_kinect.so">
-        <robotNamespace>$(arg prefix)</robotNamespace>
-        <baseline>0.2</baseline>
+      <material>Gazebo/$(arg color)</material>
+    </gazebo>
+    <gazebo reference="$(arg prefix)/camera_accel_optical_frame">
+      <gravity>true</gravity>
+      <sensor name="imu_sensor" type="imu">
         <alwaysOn>true</alwaysOn>
-        <!-- Keep this zero, update_rate in the parent <sensor> tag
- will control the frame rate. -->
-        <updateRate>0.0</updateRate>
-        <cameraName>camera_ir</cameraName>
-        <!--imageTopicName>/camera/color/image_raw</imageTopicName>
- <cameraInfoTopicName>/camera/color/camera_info</cameraInfoTopicName>
- <depthImageTopicName>/camera/depth/image_raw</depthImageTopicName>
- <depthImageCameraInfoTopicName>/camera/depth/camera_info</depthImageCameraInfoTopicName>
- <pointCloudTopicName>/camera/depth/points</pointCloudTopicName-->
-        <frameName>kinect_optical_ros_link</frameName>
-        <pointCloudCutoff>1.2</pointCloudCutoff>
-        <pointCloudCutoffMax>3.5</pointCloudCutoffMax>
-        <distortionK1>0</distortionK1>
-        <distortionK2>0</distortionK2>
-        <distortionK3>0</distortionK3>
-        <distortionT1>0</distortionT1>
-        <distortionT2>0</distortionT2>
-        <CxPrime>0</CxPrime>
-        <Cx>0</Cx>
-        <Cy>0</Cy>
-        <focalLength>0</focalLength>
-        <hackBaseline>0</hackBaseline>
-      </plugin>
-    </sensor>
-    <material>Gazebo/$(arg color)</material>
-  </gazebo>
-  <gazebo reference="$(arg prefix)/imu_link">
-    <sensor name="imu_sensor" type="imu">
-      <plugin filename="libgazebo_ros_imu_sensor.so" name="imu_plugin">
-        <robotNamespace>$(arg prefix)</robotNamespace>
-        <topicName>imu/data</topicName>
-        <bodyName>$(arg prefix)/imu_link</bodyName>
-        <updateRateHZ>100</updateRateHZ>
-        <gaussianNoise>0.01</gaussianNoise>
-        <xyzOffset>0 0 0</xyzOffset>
-        <rpyOffset>0 0 0</rpyOffset>
-        <frameName>$(arg prefix)/imu_link</frameName>
-      </plugin>
-    </sensor>
-  </gazebo>
+        <update_rate>100</update_rate>
+        <plugin filename="libgazebo_ros_imu_sensor.so" name="imu_plugin">
+          <robotNamespace>$(arg prefix)</robotNamespace>
+          <topicName>camera/imu</topicName>
+          <bodyName>$(arg prefix)/camera_accel_optical_frame</bodyName>
+          <updateRateHZ>100</updateRateHZ>
+          <gaussianNoise>0.0</gaussianNoise>
+          <xyzOffset>0 0 0</xyzOffset>
+          <rpyOffset>0 0 0</rpyOffset>
+          <frameName>$(arg prefix)/camera_accel_optical_frame</frameName>
+          <initialOrientationAsReference>false</initialOrientationAsReference>
+        </plugin>
+      </sensor>
+    </gazebo>
+  </xacro:if>
 </robot>

Commit message: Rotated Lidar frame
- The real life lidar has an orientation shift of 45 deg

File: src/swarmus_ros_description/urdf/pioneer.urdf.xacro (robot description, xacro)
@@ -10,4 +10,5 @@
   <link name="$(arg prefix)/base_footprint" />
   <link name="$(arg prefix)/base_link" />
+  <xacro:property name="M_PI" value="3.1415926535897931" />
   <!-- ================================== Links ==================================-->
   <link name="$(arg prefix)/chassis">
@@ -160,5 +161,5 @@
     <child link="$(arg prefix)/rplidar"/>
     <parent link="$(arg prefix)/chassis" />
-    <origin rpy="0 0 0" xyz="0.02378 0 0.19709"/>
+    <origin rpy="0 0 ${M_PI/4}" xyz="0.02378 0 0.19709"/>
   </joint>
   <joint name="hiveboard_joint" type="fixed">

Commit message: Updated the lidar frame and adjusted its urdf orientation

File: src/swarmus_ros_description/urdf/pioneer.urdf.xacro (robot description, xacro)
@@ -161,5 +161,5 @@
     <child link="$(arg prefix)/rplidar"/>
     <parent link="$(arg prefix)/chassis" />
-    <origin rpy="0 0 ${M_PI/4}" xyz="0.02378 0 0.19709"/>
+    <origin rpy="0 0 ${-M_PI*3/4}" xyz="0.02378 0 0.19709"/>
   </joint>
   <joint name="hiveboard_joint" type="fixed">

Commit message: Feat/swarinfo 165 camera configurations (#26)
* Initial D435i launchfile

* Added dependency

* Added state robot_publisher and the d435i bringup

- Added a namespace to add the same prefix as the main simulation robot (pioneer_0)
- Remove the camera initial reset since it slow down the boot up sequence during developpment
- Added the pointcloud for rviz visualization
- Included the d435i bringup into the main bringup
- Added the node robot_state_publisher

* Adjusted IMU frame rates

* Added D455 bringup

- Added the D455 bringup launchfile
- Added an argument to set easily the camera fps

* Fixed the FPS argument that was no changing the camera frame rate. Changed parameter to save computation power on the PI. This setup might changed but its a starting point.

* Lowered computation of camera node

- Lowered the D435i resolution
- Changed the point cloud stream_texture to have monochrome point cloud. It saves a little bit of computation

* Rotated Lidar frame 

- The real life lidar has an orientation shift of 45 deg

* Updated the lidar frame and adjusted its urdf orientation

Co-authored-by: Etienne <vile2094@usherbrooke.ca>

File: src/swarmus_ros_description/urdf/pioneer.urdf.xacro (robot description, xacro)
@@ -10,4 +10,5 @@
   <link name="$(arg prefix)/base_footprint" />
   <link name="$(arg prefix)/base_link" />
+  <xacro:property name="M_PI" value="3.1415926535897931" />
   <!-- ================================== Links ==================================-->
   <link name="$(arg prefix)/chassis">
@@ -160,5 +161,5 @@
     <child link="$(arg prefix)/rplidar"/>
     <parent link="$(arg prefix)/chassis" />
-    <origin rpy="0 0 0" xyz="0.02378 0 0.19709"/>
+    <origin rpy="0 0 ${-M_PI*3/4}" xyz="0.02378 0 0.19709"/>
   </joint>
   <joint name="hiveboard_joint" type="fixed">

Commit message: Changed gazebo parameter to reflect the real robot

File: src/swarmus_ros_description/urdf/pioneer.urdf.xacro (robot description, xacro)
@@ -11,4 +11,6 @@
   <link name="$(arg prefix)/base_link" />
   <xacro:property name="M_PI" value="3.1415926535897931" />
+  <xacro:property name="wheel_radius" value="0.0825" />
+  <xacro:property name="base_width" value="0.32" />
   <!-- ================================== Links ==================================-->
   <link name="$(arg prefix)/chassis">
@@ -25,5 +27,5 @@
     </collision>
     <collision name="caster_collision">
-      <origin rpy="0 0 0" xyz="-0.2 0 -0.12"/>
+      <origin rpy="0 0 0" xyz="-0.2 0 ${-wheel_radius - 0.05 + 0.04}"/>
       <geometry>
         <sphere radius="0.04"/>
@@ -37,5 +39,5 @@
     </visual>
     <visual name="caster_visual">
-      <origin rpy="0 0 0" xyz="-0.2 0 -0.12"/>
+      <origin rpy="0 0 0" xyz="-0.2 0 ${-wheel_radius - 0.05 + 0.04}"/>
       <geometry>
         <sphere radius="0.04"/>
@@ -52,11 +54,11 @@
       <origin rpy="0 0 0" xyz="0 0 0"/>
       <geometry>
-        <cylinder length="0.05" radius="0.11"/>
-      </geometry>
-    </collision>
-    <visual name="visual">
-      <origin rpy="0 0 0" xyz="0 0 0"/>
-      <geometry>
-        <cylinder length="0.05" radius="0.11"/>
+        <cylinder length="0.05" radius="${wheel_radius}"/>
+      </geometry>
+    </collision>
+    <visual name="visual">
+      <origin rpy="0 0 0" xyz="0 0 0"/>
+      <geometry>
+        <cylinder length="0.05" radius="${wheel_radius}"/>
       </geometry>
     </visual>
@@ -71,11 +73,11 @@
       <origin rpy="0 0 0" xyz="0 0 0"/>
       <geometry>
-        <cylinder length="0.05" radius="0.11"/>
-      </geometry>
-    </collision>
-    <visual name="visual">
-      <origin rpy="0 0 0" xyz="0 0 0"/>
-      <geometry>
-        <cylinder length="0.05" radius="0.11"/>
+        <cylinder length="0.05" radius="${wheel_radius}"/>
+      </geometry>
+    </collision>
+    <visual name="visual">
+      <origin rpy="0 0 0" xyz="0 0 0"/>
+      <geometry>
+        <cylinder length="0.05" radius="${wheel_radius}"/>
       </geometry>
     </visual>
@@ -135,6 +137,6 @@
   <!-- ================================== Joints ==================================-->
   <joint name="base_footprint_link_joint" type="fixed">
-    <origin xyz="-0.1 0 0.16" rpy="0 0 0" />
-    <parent link="$(arg prefix)/base_footprint" />
+    <origin xyz="-0.1 0 ${wheel_radius + 0.05}" rpy="0 0 0" />
+    <parent link="$(arg prefix)/base_footprint"/>
     <child link="$(arg prefix)/base_link" />
   </joint>
@@ -147,5 +149,5 @@
     <parent link="$(arg prefix)/chassis"/>
     <child link="$(arg prefix)/left_wheel"/>
-    <origin rpy="0 1.5707 1.5707" xyz="0.1 0.17 -0.05"/>
+    <origin rpy="0 1.5707 1.5707" xyz="0.1 ${base_width/2} -0.05"/>
     <axis xyz="9.00000000e-05 9.00000000e-05 1.00000000e+00"/>
     <limit effort="100.0" velocity="100"/>
@@ -154,5 +156,5 @@
     <parent link="$(arg prefix)/chassis"/>
     <child link="$(arg prefix)/right_wheel"/>
-    <origin rpy="0 1.5707 1.5707" xyz="0.1 -0.17 -0.05"/>
+    <origin rpy="0 1.5707 1.5707" xyz="0.1 ${-base_width/2}  -0.05"/>
     <axis xyz="9.00000000e-05 9.00000000e-05 1.00000000e+00"/>
     <limit effort="100.0" velocity="100"/>
@@ -209,7 +211,7 @@
         <leftJoint>left_wheel_hinge</leftJoint>
         <rightJoint>right_wheel_hinge</rightJoint>
-        <wheelSeparation>0.34</wheelSeparation>
-        <wheelDiameter>0.22</wheelDiameter>
-        <wheelAcceleration>1</wheelAcceleration>
+        <wheelSeparation>${base_width}</wheelSeparation>
+        <wheelDiameter>${2*wheel_radius}</wheelDiameter>
+        <wheelAcceleration>0.6</wheelAcceleration>
         <wheelTorque>10</wheelTorque>
         <rosDebugLevel>true</rosDebugLevel>
